File: item_2022_Motherboard_04_V8.brd (EAGLE design)
At the start: 160 x 100 mm, 126 parts, among them IC1 MCP602SN, IC2 LD117AS33TR, IC3 MCP1525TO, IC4 MCP6S26, IC5 MCP6004SO, IC6 MCP6004SO, IC7 MCP3204SL, IC8 LM336LP, IC9 MCP6004SO, U1 ESP32-DEVKITC-32D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

Commit message: loghi
Parts:
- added U$1: (no value), ITEM_Loghi:BASSA
- added U$2: (no value), ITEM_Loghi:UDINE
- added U$3: (no value), ITEM_Loghi:DANIELI
- moved GND 9.97 mm to (145.9, 84.4)
- moved TP7 0.64 mm to (121.3, 87.0)
Routing:
- net GND: track 950.3 -> 940.9 mm
- net VSPI_MISO: track 263.1 -> 255.8 mm
- net +5V: track 312.9 -> 313.6 mm
Other:
- board text added: "D.L.23"
- board text added: "DANIELI BUTTRIO"
- board text added: "ISIS BASSA FRIULANA"
- board text added: "ISIS MALIGNANI"
- board text added: "PROGETTO ITEM"
- board text removed: "ITEM 1^ ED."
Changed lines of the file:
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@@
 <?xml version="1.0" encoding="utf-8"?>
 <!DOCTYPE eagle SYSTEM "eagle.dtd">
-<eagle version="9.6.2">
+<eagle version="7.7.0">
 <drawing>
 <settings>
 <setting alwaysvectorfont="no"/>
-<setting keepoldvectorfont="yes"/>
 <setting verticaltext="up"/>
 </settings>
@@
 <hole x="84.45" y="94.28" drill="3.2"/>
 <text x="53.34" y="18.415" size="1.9304" layer="25" align="center">ISIS BASSA FRIULANA - A.S.2022-23</text>
-<text x="53.975" y="14.605" size="1.9304" layer="25" align="center">ITEM 1^ ED.</text>
+<text x="53.975" y="14.605" size="1.9304" layer="25" align="center">PROGETTO ITEM</text>
 <text x="2.54" y="52.705" size="1.9304" layer="25" rot="R90" align="center">MOTHERBOARD</text>
 <text x="85.725" y="11.43" size="1.9304" layer="25" align="center">ACCEL_0</text>
@@
 <dimension x1="0" y1="100" x2="3" y2="97" x3="1.5" y3="105" textsize="1.778" layer="25" dtype="horizontal"/>
 <dimension x1="77.4954" y1="7.5438" x2="70.9" y2="0" x3="65" y3="3.7719" textsize="1.778" layer="47" dtype="vertical"/>
+<text x="127.9525" y="86.6775" size="1.016" layer="21" align="center">ISIS
+BASSA FRIULANA</text>
+<text x="138.43" y="86.6775" size="1.016" layer="21" align="center">ISIS
+MALIGNANI</text>
+<text x="149.5425" y="86.6775" size="1.016" layer="21" align="center">DANIELI
+BUTTRIO</text>
+<text x="40.3225" y="40.9575" size="1.27" layer="21" align="center">D.L.23</text>
 </plain>
 <attributes>
@@
 <param name="dpMaxLengthDifference" value="10mm"/>
 <param name="dpGapFactor" value="2.5"/>
+<param name="checkGrid" value="0"/>
 <param name="checkAngle" value="0"/>
 <param name="checkFont" value="1"/>
 <param name="checkRestrict" value="1"/>
-<param name="checkStop" value="0"/>
-<param name="checkValues" value="0"/>
-<param name="checkNames" value="1"/>
-<param name="checkWireStubs" value="1"/>
-<param name="checkPolygonWidth" value="0"/>
 <param name="useDiameter" value="13"/>
 <param name="maxErrors" value="50"/>
@@
 <attribute name="VALUE" x="142.367" y="65.405" size="1.27" layer="27" rot="R90"/>
 </element>
-<element name="GND" library="testpad" package="TP18SQ" value="TPTP18SQ" x="153.79" y="90.39" smashed="yes">
-<attribute name="NAME" x="152.8901" y="91.34" size="1.27" layer="25"/>
-<attribute name="TP_SIGNAL_NAME" value="" x="153.79" y="87.85" size="1" layer="37"/>
-<attribute name="VALUE" x="152.901" y="89.374" size="0.0254" layer="27"/>
+<element name="GND" library="testpad" package="TP18SQ" value="TPTP18SQ" x="145.8525" y="84.3575" smashed="yes">
+<attribute name="NAME" x="142.4126" y="81.4975" size="1.27" layer="25"/>
+<attribute name="TP_SIGNAL_NAME" value="" x="145.8525" y="81.8175" size="1" layer="37"/>
+<attribute name="VALUE" x="144.9635" y="83.3415" size="0.0254" layer="27"/>
 </element>
 <element name="GND36" library="testpad" package="TP18SQ" value="TPTP18SQ" x="149.4" y="10.0625" smashed="yes">
@@
 <attribute name="VALUE" x="148.511" y="9.0465" size="0.0254" layer="27"/>
 </element>
-<element name="TP7" library="testpad" package="TP16R" value="TPTP16R" x="121.92" y="86.995" smashed="yes">
-<attribute name="NAME" x="121.1199" y="87.8449" size="1.27" layer="25"/>
-<attribute name="TP_SIGNAL_NAME" value="" x="121.92" y="84.455" size="1" layer="37"/>
-<attribute name="VALUE" x="121.285" y="86.233" size="0.0254" layer="27"/>
+<element name="TP7" library="testpad" package="TP16R" value="TPTP16R" x="121.285" y="86.995" smashed="yes">
+<attribute name="NAME" x="117.3099" y="85.3049" size="1.27" layer="25"/>
+<attribute name="TP_SIGNAL_NAME" value="" x="121.285" y="84.455" size="1" layer="37"/>
+<attribute name="VALUE" x="120.65" y="86.233" size="0.0254" layer="27"/>
 </element>
 <element name="TP8" library="testpad" package="TP16R" value="TPTP16R" x="121.285" y="59.055" smashed="yes">
@@
 <attribute name="VALUE" x="24.13" y="83.82" size="1.27" layer="27" rot="R90"/>
 </element>
+<element name="U$1" library="ITEM_Loghi" package="BASSA" value="" x="122.2375" y="87.63"/>
+<element name="U$2" library="ITEM_Loghi" package="UDINE" value="" x="133.35" y="87.63"/>
+<element name="U$3" library="ITEM_Loghi" package="DANIELI" value="" x="144.145" y="88.5825"/>
 </elements>
 <signals>
@@
 <wire x1="150.2664" y1="72.9996" x2="150.175" y2="73.025" width="0.4064" layer="1"/>
 <wire x1="150.4188" y1="70.5612" x2="150.495" y2="70.3834" width="0.4064" layer="1"/>
-<wire x1="153.7716" y1="88.6968" x2="153.7716" y2="90.3732" width="0.4064" layer="1"/>
-<wire x1="146.6088" y1="81.534" x2="153.7716" y2="88.6968" width="0.4064" layer="1"/>
-<wire x1="146.6088" y1="76.962" x2="146.6088" y2="81.534" width="0.4064" layer="1"/>
-<wire x1="150.114" y1="73.4568" x2="146.6088" y2="76.962" width="0.4064" layer="1"/>
+<wire x1="145.8341" y1="82.3468" x2="145.8341" y2="84.0232" width="0.4064" layer="1"/>
+<wire x1="145.9738" y1="81.8515" x2="145.8341" y2="82.3468" width="0.4064" layer="1"/>
+<wire x1="145.9738" y1="77.2795" x2="145.9738" y2="81.8515" width="0.4064" layer="1"/>
+<wire x1="150.114" y1="73.4568" x2="145.9738" y2="77.2795" width="0.4064" layer="1"/>
 <wire x1="150.114" y1="73.152" x2="150.114" y2="73.4568" width="0.4064" layer="1"/>
-<wire x1="153.7716" y1="90.3732" x2="153.79" y2="90.39" width="0.4064" layer="1"/>
+<wire x1="145.8341" y1="84.0232" x2="145.8525" y2="84.3575" width="0.4064" layer="1"/>
 <wire x1="150.114" y1="73.152" x2="150.175" y2="73.025" width="0.4064" layer="1"/>
 <wire x1="155.448" y1="65.3796" x2="155.448" y2="64.3128" width="0.4064" layer="1"/>
@@
 <wire x1="150.5712" y1="69.342" x2="150.4188" y2="69.342" width="0.4064" layer="1"/>
 <wire x1="145.542" y1="82.4484" x2="125.2728" y2="82.4484" width="0.4064" layer="1"/>
-<wire x1="146.4564" y1="81.534" x2="145.542" y2="82.4484" width="0.4064" layer="1"/>
+<wire x1="145.8214" y1="82.169" x2="145.542" y2="82.4484" width="0.4064" layer="1"/>
 <wire x1="125.2728" y1="82.4484" x2="125.24" y2="82.55" width="0.4064" layer="1"/>
-<wire x1="146.4564" y1="81.534" x2="146.6088" y2="81.534" width="0.4064" layer="1"/>
+<wire x1="145.8214" y1="82.169" x2="145.9738" y2="81.8515" width="0.4064" layer="1"/>
 <wire x1="106.3752" y1="95.4024" x2="106.0704" y2="95.4024" width="0.4064" layer="1"/>
 <wire x1="117.9576" y1="83.82" x2="108.4326" y2="93.345" width="0.4064" layer="1"/>
@@
 <via x="139.7" y="74.6125" extent="1-16" drill="0.6"/>
 <via x="152.0825" y="97.79" extent="1-16" drill="0.6"/>
-<via x="148.59" y="95.5675" extent="1-16" drill="0.6"/>
+<via x="143.1925" y="95.885" extent="1-16" drill="0.6"/>
 <via x="154.94" y="86.0425" extent="1-16" drill="0.6"/>
 <via x="121.285" y="95.5675" extent="1-16" drill="0.6"/>
@@
 <wire x1="54.7116" y1="23.3172" x2="54.61" y2="22.5425" width="0.4064" layer="1"/>
 <wire x1="54.7116" y1="27.1272" x2="54.6875" y2="27.33" width="0.4064" layer="1"/>
-<wire x1="25.4508" y1="45.1104" x2="16.6116" y2="45.1104" width="0.8128" layer="1"/>
+<wire x1="29.5275" y1="45.1104" x2="16.6116" y2="45.1104" width="0.8128" layer="1"/>
 <wire x1="44.8056" y1="25.1206" x2="32.0675" y2="38.1" width="0.8128" layer="1"/>
 <wire x1="32.0675" y1="38.1" x2="32.0675" y2="42.5704" width="0.8128" layer="1"/>
 <wire x1="32.0675" y1="42.5704" x2="29.5275" y2="45.1104" width="0.8128" layer="1"/>
-<wire x1="29.5275" y1="45.1104" x2="25.4508" y2="45.1104" width="0.8128" layer="1"/>
 <wire x1="54.7116" y1="25.1206" x2="44.8056" y2="25.1206" width="0.8128" layer="1"/>
 <wire x1="16.6116" y1="45.1104" x2="16.51" y2="45.16" width="0.4064" layer="1"/>
@@
 <wire x1="117.0432" y1="87.0204" x2="121.92" y2="87.0204" width="0.4064" layer="1"/>
 <wire x1="108.6612" y1="95.4024" x2="117.0432" y2="87.0204" width="0.4064" layer="1"/>
-<wire x1="121.92" y1="87.0204" x2="121.92" y2="86.995" width="0.4064" layer="1"/>
+<wire x1="121.92" y1="87.0204" x2="121.285" y2="86.995" width="0.4064" layer="1"/>
 <wire x1="108.6612" y1="95.4024" x2="108.57" y2="95.55" width="0.4064" layer="1"/>
 <wire x1="96.774" y1="60.0456" x2="96.774" y2="57.15" width="0.4064" layer="1"/>
@@
 <wire x1="149.9616" y1="76.2" x2="153.0096" y2="73.152" width="0.254" layer="1"/>
 <wire x1="149.9616" y1="83.9724" x2="149.9616" y2="76.2" width="0.254" layer="1"/>
-<wire x1="155.1432" y1="89.154" x2="149.9616" y2="83.9724" width="0.254" layer="1"/>
-<wire x1="155.1432" y1="91.5924" x2="155.1432" y2="89.154" width="0.254" layer="1"/>
-<wire x1="149.1996" y1="97.536" x2="155.1432" y2="91.5924" width="0.254" layer="1"/>
-<wire x1="97.9932" y1="97.536" x2="149.1996" y2="97.536" width="0.254" layer="1"/>
+<wire x1="150.0632" y1="89.154" x2="149.9616" y2="83.9724" width="0.254" layer="1"/>
+<wire x1="150.0632" y1="91.5924" x2="150.0632" y2="89.154" width="0.254" layer="1"/>
+<wire x1="144.1196" y1="97.536" x2="150.0632" y2="91.5924" width="0.254" layer="1"/>
+<wire x1="97.9932" y1="97.536" x2="144.1196" y2="97.536" width="0.254" layer="1"/>
 <wire x1="97.0788" y1="96.6216" x2="97.9932" y2="97.536" width="0.254" layer="1"/>
 <wire x1="97.0788" y1="94.3356" x2="97.0788" y2="96.6216" width="0.254" layer="1"/>
@@
 </signal>
 </signals>
-<mfgpreviewcolors>
-<mfgpreviewcolor name="soldermaskcolor" color="0xC8008000"/>
-<mfgpreviewcolor name="silkscreencolor" color="0xFFFEFEFE"/>
-<mfgpreviewcolor name="backgroundcolor" color="0xFF282828"/>
-<mfgpreviewcolor name="coppercolor" color="0xFFFFBF00"/>
-<mfgpreviewcolor name="substratecolor" color="0xFF786E46"/>
-</mfgpreviewcolors>
 </board>
 </drawing>
+<compatibility>
+<note version="6.3" minversion="6.2.2" severity="warning">
+Since Version 6.2.2 text objects can contain more than one line,
+which will not be processed correctly with this version.
+</note>
+</compatibility>
 </eagle>

Commit message: corretto layer 21
Routing:
- net GND: vias 121 -> 122
Changed lines of the file:
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@@
 <layer number="37" name="tTest" color="7" fill="1" visible="no" active="yes"/>
 <layer number="38" name="bTest" color="7" fill="1" visible="no" active="yes"/>
-<layer number="39" name="tKeepout" color="4" fill="11" visible="yes" active="yes"/>
-<layer number="40" name="bKeepout" color="1" fill="11" visible="yes" active="yes"/>
-<layer number="41" name="tRestrict" color="4" fill="10" visible="yes" active="yes"/>
-<layer number="42" name="bRestrict" color="1" fill="10" visible="yes" active="yes"/>
+<layer number="39" name="tKeepout" color="4" fill="11" visible="no" active="yes"/>
+<layer number="40" name="bKeepout" color="1" fill="11" visible="no" active="yes"/>
+<layer number="41" name="tRestrict" color="4" fill="10" visible="no" active="yes"/>
+<layer number="42" name="bRestrict" color="1" fill="10" visible="no" active="yes"/>
 <layer number="43" name="vRestrict" color="2" fill="10" visible="no" active="yes"/>
 <layer number="44" name="Drills" color="7" fill="1" visible="yes" active="yes"/>
 <layer number="45" name="Holes" color="7" fill="1" visible="yes" active="yes"/>
 <layer number="46" name="Milling" color="3" fill="1" visible="no" active="yes"/>
-<layer number="47" name="Measures" color="7" fill="1" visible="yes" active="yes"/>
-<layer number="48" name="Document" color="7" fill="1" visible="no" active="yes"/>
+<layer number="47" name="Measures" color="7" fill="1" visible="no" active="yes"/>
+<layer number="48" name="Document" color="7" fill="1" visible="yes" active="yes"/>
 <layer number="49" name="Reference" color="7" fill="1" visible="no" active="yes"/>
 <layer number="51" name="tDocu" color="7" fill="1" visible="yes" active="yes"/>
@@
 <text x="8.255" y="45.4025" size="0.6096" layer="21">GND</text>
 <text x="28.8925" y="95.5675" size="1.778" layer="25" align="center">ANTENNA</text>
-<dimension x1="0" y1="0" x2="85.09" y2="2.54" x3="42.545" y3="-10" textsize="1.778" layer="25" dtype="horizontal"/>
-<dimension x1="0" y1="0" x2="107.95" y2="2.54" x3="53.975" y3="-15" textsize="1.778" layer="25" dtype="horizontal"/>
-<dimension x1="3" y1="1.25" x2="3" y2="4.75" x3="-5" y3="3" textsize="1.778" layer="25" dtype="diameter"/>
-<dimension x1="0" y1="0" x2="160" y2="11" x3="80" y3="-20" textsize="1.778" layer="25" dtype="horizontal"/>
-<dimension x1="160" y1="0" x2="153.7" y2="100" x3="166.3" y3="50" textsize="1.778" layer="25" dtype="vertical"/>
-<dimension x1="0" y1="100" x2="3" y2="97" x3="-10" y3="98.5" textsize="1.778" layer="25" dtype="vertical"/>
-<dimension x1="0" y1="100" x2="3" y2="97" x3="1.5" y3="105" textsize="1.778" layer="25" dtype="horizontal"/>
+<dimension x1="0" y1="0" x2="85.09" y2="2.54" x3="42.545" y3="-10" textsize="1.778" layer="47" dtype="horizontal"/>
+<dimension x1="0" y1="0" x2="107.95" y2="2.54" x3="53.975" y3="-15" textsize="1.778" layer="47" dtype="horizontal"/>
+<dimension x1="3" y1="1.25" x2="3" y2="4.75" x3="-5" y3="3" textsize="1.778" layer="47" dtype="diameter"/>
+<dimension x1="0" y1="0" x2="160" y2="11" x3="80" y3="-20" textsize="1.778" layer="47" dtype="horizontal"/>
+<dimension x1="160" y1="0" x2="153.7" y2="100" x3="166.3" y3="50" textsize="1.778" layer="47" dtype="vertical"/>
+<dimension x1="0" y1="100" x2="3" y2="97" x3="-10" y3="98.5" textsize="1.778" layer="47" dtype="vertical"/>
+<dimension x1="0" y1="100" x2="3" y2="97" x3="1.5" y3="105" textsize="1.778" layer="47" dtype="horizontal"/>
 <dimension x1="77.4954" y1="7.5438" x2="70.9" y2="0" x3="65" y3="3.7719" textsize="1.778" layer="47" dtype="vertical"/>
 <text x="127.9525" y="86.6775" size="1.016" layer="21" align="center">ISIS
@@
 </element>
 <element name="U2" library="ADS1256" package="ADS1256_BOARD" value="ADS1256_BOARD" x="100.95" y="67.61" smashed="yes" rot="MR90">
-<attribute name="NAME" x="118.73" y="37.13" size="1.27" layer="22" font="vector" rot="MR90" align="center-left"/>
-<attribute name="VALUE" x="80.63" y="37.13" size="1.27" layer="22" font="vector" rot="MR90" align="center-left"/>
+<attribute name="NAME" x="118.73" y="37.13" size="1.27" layer="21" font="vector" rot="R90" align="center-left"/>
+<attribute name="VALUE" x="80.63" y="37.13" size="1.27" layer="21" font="vector" rot="R90" align="center-left"/>
 </element>
 <element name="U3" library="ssd1306oled" package="128X64" value="SSD1306_128X64" x="16.25" y="27.725" smashed="yes"/>
@@
 <attribute name="VALUE" x="24.13" y="83.82" size="1.27" layer="27" rot="R90"/>
 </element>
-<element name="U$1" library="ITEM_Loghi" package="BASSA" value="" x="122.2375" y="87.63"/>
-<element name="U$2" library="ITEM_Loghi" package="UDINE" value="" x="133.35" y="87.63"/>
-<element name="U$3" library="ITEM_Loghi" package="DANIELI" value="" x="144.145" y="88.5825"/>
+<element name="U$1" library="ITEM_Loghi" package="BASSA" value="" x="122.2375" y="87.63" smashed="yes"/>
+<element name="U$2" library="ITEM_Loghi" package="UDINE" value="" x="133.35" y="87.63" smashed="yes"/>
+<element name="U$3" library="ITEM_Loghi" package="DANIELI" value="" x="144.145" y="88.5825" smashed="yes"/>
 </elements>
 <signals>
@@
 <via x="74.93" y="93.6625" extent="1-16" drill="0.6"/>
 <via x="74.6125" y="81.28" extent="1-16" drill="0.6"/>
-<via x="81.5975" y="81.28" extent="1-16" drill="0.6"/>
+<via x="81.28" y="81.28" extent="1-16" drill="0.6"/>
 <via x="81.28" y="77.47" extent="1-16" drill="0.6"/>
 <via x="74.6125" y="77.47" extent="1-16" drill="0.6"/>
@@
 <via x="74.295" y="59.055" extent="1-16" drill="0.6"/>
 <via x="83.185" y="55.88" extent="1-16" drill="0.6"/>
-<via x="89.2175" y="53.34" extent="1-16" drill="0.6"/>
-<via x="84.7725" y="48.26" extent="1-16" drill="0.6"/>
-<via x="95.25" y="53.0225" extent="1-16" drill="0.6"/>
-<via x="103.1875" y="53.0225" extent="1-16" drill="0.6"/>
-<via x="110.49" y="53.0225" extent="1-16" drill="0.6"/>
+<via x="88.9" y="53.6575" extent="1-16" drill="0.6"/>
+<via x="86.36" y="48.895" extent="1-16" drill="0.6"/>
+<via x="95.25" y="53.6575" extent="1-16" drill="0.6"/>
+<via x="103.1875" y="53.6575" extent="1-16" drill="0.6"/>
+<via x="110.8075" y="53.975" extent="1-16" drill="0.6"/>
 <via x="110.49" y="59.3725" extent="1-16" drill="0.6"/>
 <via x="117.475" y="59.69" extent="1-16" drill="0.6"/>
@@
 <via x="48.895" y="77.47" extent="1-16" drill="0.6"/>
 <via x="128.27" y="66.3575" extent="1-16" drill="0.6"/>
+<via x="116.84" y="91.1225" extent="1-16" drill="0.6"/>
+<wire x1="121.285" y1="95.5675" x2="116.84" y2="91.1225" width="0" layer="19" extent="1-1"/>
 </signal>
 <signal name="+5V" class="1">
@@
 <wire x1="16.6116" y1="90.8304" x2="16.51" y2="90.88" width="0.3048" layer="1"/>
 </signal>
-<signal name="N$44">
-<via x="117.475" y="91.44" extent="1-16" drill="0.6"/>
-</signal>
 </signals>
