File: item_2022_Motherboard_04_V8.brd (EAGLE design)
At the start: 160 x 100 mm, 129 parts, among them IC1 MCP602SN, IC2 LD117AS33TR, IC3 MCP1525TO, IC4 MCP6S26, IC5 MCP6004SO, IC6 MCP6004SO, IC7 MCP3204SL, IC8 LM336LP, IC9 MCP6004SO, U1 ESP32-DEVKITC-32D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

Commit message: cambio package elettrolitici smd
Parts:
- added C31: 220uF/16V, rcl@1:E3,5-10
- C14: value 10uF / 16V -> 10uF/16V; device rcl_LargePads:PANASONIC_C -> rcl@1:E2,5-6
- C4: device rcl@1:E3,5-8 -> rcl@1:E2,5-6
- moved C14 0.45 mm to (122.9, 82.2), turned to 0 degrees
Connections:
- net +5V: now also C31.+
- net GND: now also C31.-
Routing:
- net GND: track 940.9 -> 943.0 mm
- net +3V3: track 266.8 -> 267.6 mm
Other:
- board text added: "PROGETTO ITEM - A.S.2022-23"
- board text removed: "ISIS BASSA FRIULANA - A.S.2022-23"
- board text removed: "PROGETTO ITEM"
Changed lines of the file:
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@@
 <?xml version="1.0" encoding="utf-8"?>
 <!DOCTYPE eagle SYSTEM "eagle.dtd">
-<eagle version="9.6.2">
+<eagle version="7.7.0">
 <drawing>
 <settings>
 <setting alwaysvectorfont="no"/>
-<setting keepoldvectorfont="yes"/>
 <setting verticaltext="up"/>
 </settings>
@@
 <hole x="114.92" y="94.28" drill="3.2"/>
 <hole x="84.45" y="94.28" drill="3.2"/>
-<text x="53.34" y="18.415" size="1.9304" layer="25" align="center">ISIS BASSA FRIULANA - A.S.2022-23</text>
-<text x="53.975" y="14.605" size="1.9304" layer="25" align="center">PROGETTO ITEM</text>
+<text x="47.625" y="18.415" size="1.9304" layer="25" align="center">ISIS BASSA FRIULANA</text>
+<text x="53.0225" y="14.605" size="1.9304" layer="25" align="center">PROGETTO ITEM - A.S.2022-23</text>
 <text x="2.54" y="52.705" size="1.9304" layer="25" rot="R90" align="center">MOTHERBOARD</text>
 <text x="85.725" y="11.43" size="1.9304" layer="25" align="center">ACCEL_0</text>
@@
 </class>
 </classes>
-<designrules name="default">
+<designrules name="default *">
 <description language="de">&lt;b&gt;EAGLE Design Rules&lt;/b&gt;
 &lt;p&gt;
@@
 <param name="mdSmdStop" value="0mil"/>
 <param name="msWidth" value="10mil"/>
-<param name="msDrill" value="24mil"/>
+<param name="msDrill" value="0.2mm"/>
 <param name="msMicroVia" value="9.99mm"/>
 <param name="msBlindViaRatio" value="0.5"/>
@@
 <param name="dpMaxLengthDifference" value="10mm"/>
 <param name="dpGapFactor" value="2.5"/>
+<param name="checkGrid" value="0"/>
 <param name="checkAngle" value="0"/>
 <param name="checkFont" value="1"/>
 <param name="checkRestrict" value="1"/>
-<param name="checkStop" value="0"/>
-<param name="checkValues" value="0"/>
-<param name="checkNames" value="1"/>
-<param name="checkWireStubs" value="1"/>
-<param name="checkPolygonWidth" value="0"/>
 <param name="useDiameter" value="13"/>
 <param name="maxErrors" value="50"/>
@@
 <attribute name="VALUE" x="60.0025" y="29.48" size="1.016" layer="27" rot="R90"/>
 </element>
-<element name="C4" library="rcl@1" package="E3,5-8" value="10uF/16V" x="43.815" y="30.48" smashed="yes" rot="R270">
+<element name="C4" library="rcl@1" package="E2,5-6" value="10uF/16V" x="43.815" y="30.48" smashed="yes" rot="R270">
 <attribute name="NAME" x="46.609" y="27.178" size="1.27" layer="25" ratio="10" rot="R270"/>
 <attribute name="VALUE" x="40.767" y="32.766" size="1.27" layer="27" ratio="10" rot="R270"/>
@@
 <attribute name="VALUE" x="142.875" y="48.895" size="1.27" layer="27"/>
 </element>
-<element name="C14" library="rcl_LargePads" package="PANASONIC_C" value="10uF / 16V" x="123.19" y="82.55" smashed="yes" rot="R180">
-<attribute name="NAME" x="125.79" y="79.8" size="1.016" layer="25" rot="R180"/>
-<attribute name="VALUE" x="125.84" y="86.325" size="1.016" layer="27" rot="R180"/>
-</element>
 <element name="R10" library="rcl_LargePads" package="R0805" value="6.8k" x="136.525" y="73.025" smashed="yes" rot="R180">
 <attribute name="NAME" x="137.16" y="71.755" size="1.27" layer="25" rot="R180"/>
@@
 <element name="U$2" library="ITEM_Loghi" package="UDINE" value="" x="133.35" y="87.63" smashed="yes"/>
 <element name="U$3" library="ITEM_Loghi" package="DANIELI" value="" x="144.145" y="88.5825" smashed="yes"/>
+<element name="C14" library="rcl@1" package="E2,5-6" value="10uF/16V" x="122.8725" y="82.2325"/>
+<element name="C31" library="rcl@1" package="E3,5-10" value="220uF/16V" x="65.0875" y="22.86"/>
 </elements>
 <signals>
@@
 <wire x1="42.3672" y1="30.7848" x2="42.3672" y2="26.3652" width="0.4064" layer="16"/>
 <wire x1="43.7388" y1="32.1564" x2="42.3672" y2="30.7848" width="0.4064" layer="16"/>
-<wire x1="43.7388" y1="32.1564" x2="43.815" y2="32.258" width="0.4064" layer="16"/>
+<wire x1="43.7388" y1="32.1564" x2="43.815" y2="31.75" width="0.4064" layer="16"/>
 <wire x1="12.4968" y1="34.1376" x2="12.4968" y2="40.386" width="0.4064" layer="1"/>
 <wire x1="30.48" y1="16.1544" x2="12.4968" y2="34.1376" width="0.4064" layer="1"/>
@@
 <wire x1="43.8912" y1="32.3088" x2="45.1104" y2="33.528" width="0.4064" layer="1"/>
 <wire x1="52.2732" y1="33.528" x2="52.3875" y2="33.63" width="0.4064" layer="1"/>
-<wire x1="43.8912" y1="32.3088" x2="43.815" y2="32.258" width="0.4064" layer="1"/>
+<wire x1="43.8912" y1="32.3088" x2="43.815" y2="31.75" width="0.4064" layer="1"/>
 <wire x1="148.1328" y1="70.5612" x2="148.1328" y2="72.9996" width="0.4064" layer="1"/>
 <wire x1="147.955" y1="70.3834" x2="148.1328" y2="70.5612" width="0.4064" layer="1"/>
@@
 <contactref element="IC3" pad="1"/>
 <contactref element="C12" pad="2"/>
-<contactref element="C14" pad="-"/>
 <contactref element="C13" pad="2"/>
 <contactref element="IC5" pad="11"/>
@@
 <wire x1="49.0728" y1="28.6512" x2="43.8912" y2="28.6512" width="0.4064" layer="1"/>
 <wire x1="49.9872" y1="27.7368" x2="49.0728" y2="28.6512" width="0.4064" layer="1"/>
-<wire x1="43.8912" y1="28.6512" x2="43.815" y2="28.702" width="0.4064" layer="1"/>
+<wire x1="43.8912" y1="28.6512" x2="43.815" y2="29.21" width="0.4064" layer="1"/>
 <wire x1="49.9872" y1="27.7368" x2="50.0875" y2="27.33" width="0.4064" layer="1"/>
 <wire x1="35.56" y1="11.43" x2="33.02" y2="11.43" width="0.4064" layer="1"/>
@@
 <wire x1="43.7388" y1="12.0396" x2="43.7388" y2="28.6512" width="0.4064" layer="16"/>
 <wire x1="43.2816" y1="11.5824" x2="43.7388" y2="12.0396" width="0.4064" layer="16"/>
-<wire x1="43.7388" y1="28.6512" x2="43.815" y2="28.702" width="0.4064" layer="16"/>
+<wire x1="43.7388" y1="28.6512" x2="43.815" y2="29.21" width="0.4064" layer="16"/>
 <wire x1="43.2816" y1="11.5824" x2="43.18" y2="11.43" width="0.4064" layer="16"/>
 <wire x1="33.0708" y1="11.2776" x2="33.0708" y2="8.9916" width="0.4064" layer="1"/>
@@
 <wire x1="145.542" y1="82.4484" x2="125.2728" y2="82.4484" width="0.4064" layer="1"/>
 <wire x1="145.8214" y1="82.169" x2="145.542" y2="82.4484" width="0.4064" layer="1"/>
-<wire x1="125.2728" y1="82.4484" x2="125.24" y2="82.55" width="0.4064" layer="1"/>
 <wire x1="145.8214" y1="82.169" x2="145.9738" y2="81.8515" width="0.4064" layer="1"/>
 <wire x1="106.3752" y1="95.4024" x2="106.0704" y2="95.4024" width="0.4064" layer="1"/>
@@
 <wire x1="125.1204" y1="82.6008" x2="123.9012" y2="83.82" width="0.4064" layer="1"/>
 <wire x1="106.0704" y1="95.4024" x2="106.03" y2="95.55" width="0.4064" layer="1"/>
-<wire x1="125.1204" y1="82.6008" x2="125.24" y2="82.55" width="0.4064" layer="1"/>
 <wire x1="88.392" y1="29.718" x2="86.7156" y2="29.718" width="0.4064" layer="1"/>
 <wire x1="90.678" y1="27.432" x2="88.392" y2="29.718" width="0.4064" layer="1"/>
@@
 <via x="128.27" y="66.3575" extent="1-16" drill="0.6"/>
 <via x="116.84" y="91.1225" extent="1-16" drill="0.6"/>
+<contactref element="C31" pad="-"/>
+<contactref element="C14" pad="-"/>
+<wire x1="124.1425" y1="82.2325" x2="125.1204" y2="82.2325" width="0.3048" layer="1"/>
+<wire x1="125.1204" y1="82.2325" x2="125.1204" y2="82.6008" width="0.3048" layer="1"/>
 </signal>
 <signal name="+5V" class="1">
@@
 <via x="124.0536" y="49.53" extent="1-16" drill="0.6096"/>
 <via x="90.678" y="49.9872" extent="1-16" drill="0.6096"/>
+<contactref element="C31" pad="+"/>
+<wire x1="63.373" y1="22.6822" x2="63.373" y2="22.7965" width="0.4064" layer="16"/>
+<wire x1="63.373" y1="22.7965" x2="63.3095" y2="22.86" width="0.4064" layer="16"/>
 </signal>
 <signal name="HSPI_SCK" class="2">
@@
 <contactref element="R44" pad="1"/>
 <contactref element="IC3" pad="2"/>
-<contactref element="C14" pad="+"/>
 <contactref element="R10" pad="2"/>
 <contactref element="IC9" pad="5"/>
@@
 <wire x1="135.4836" y1="72.9996" x2="135.575" y2="73.025" width="0.3048" layer="1"/>
 <wire x1="135.3312" y1="69.9516" x2="135.255" y2="69.91" width="0.3048" layer="1"/>
-<wire x1="121.158" y1="80.1624" x2="121.158" y2="82.4484" width="0.3048" layer="1"/>
+<wire x1="121.158" y1="80.1624" x2="121.158" y2="82.2325" width="0.3048" layer="1"/>
 <wire x1="123.1392" y1="78.1812" x2="121.158" y2="80.1624" width="0.3048" layer="1"/>
-<wire x1="121.158" y1="82.4484" x2="121.14" y2="82.55" width="0.3048" layer="1"/>
 <wire x1="123.1392" y1="78.1812" x2="123.19" y2="78.105" width="0.3048" layer="1"/>
 <wire x1="135.636" y1="76.0476" x2="135.636" y2="73.152" width="0.3048" layer="1"/>
@@
 <wire x1="123.2916" y1="67.6656" x2="123.19" y2="67.6275" width="0.3048" layer="16"/>
 <wire x1="123.2916" y1="78.0288" x2="123.19" y2="78.105" width="0.3048" layer="16"/>
+<contactref element="C14" pad="+"/>
+<wire x1="121.6025" y1="82.2325" x2="121.158" y2="82.2325" width="0.3048" layer="1"/>
 </signal>
 <signal name="+2.5V">
@@
 </signal>
 </signals>
-<mfgpreviewcolors>
-<mfgpreviewcolor name="soldermaskcolor" color="0xC8008000"/>
-<mfgpreviewcolor name="silkscreencolor" color="0xFFFEFEFE"/>
-<mfgpreviewcolor name="backgroundcolor" color="0xFF282828"/>
-<mfgpreviewcolor name="coppercolor" color="0xFFFFBF00"/>
-<mfgpreviewcolor name="substratecolor" color="0xFF786E46"/>
-</mfgpreviewcolors>
+<errors>
+</errors>
 </board>
 </drawing>

Commit message: migliorate piste su D1
Routing:
- net EXT_+5V: track 12.8 -> 11.6 mm
Changed lines of the file:
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@@
 <setting verticaltext="up"/>
 </settings>
-<grid distance="0.0125" unitdist="inch" unit="inch" style="lines" multiple="2" display="yes" altdistance="0.025" altunitdist="inch" altunit="inch"/>
+<grid distance="0.0125" unitdist="inch" unit="mm" style="lines" multiple="2" display="yes" altdistance="0.025" altunitdist="inch" altunit="inch"/>
 <layers>
 <layer number="1" name="Top" color="4" fill="1" visible="yes" active="yes"/>
@@
 <layer number="45" name="Holes" color="7" fill="1" visible="no" active="yes"/>
 <layer number="46" name="Milling" color="3" fill="1" visible="no" active="yes"/>
-<layer number="47" name="Measures" color="7" fill="1" visible="no" active="yes"/>
+<layer number="47" name="Measures" color="7" fill="1" visible="yes" active="yes"/>
 <layer number="48" name="Document" color="7" fill="1" visible="no" active="yes"/>
 <layer number="49" name="Reference" color="7" fill="1" visible="no" active="yes"/>
@@
 <wire x1="54.7116" y1="27.432" x2="54.6875" y2="27.33" width="0.4064" layer="1"/>
 <wire x1="54.7116" y1="27.1272" x2="54.7116" y2="25.1206" width="0.8128" layer="1"/>
-<wire x1="54.7116" y1="25.1206" x2="54.7116" y2="23.3172" width="0.8128" layer="1"/>
-<wire x1="54.7116" y1="23.3172" x2="54.61" y2="22.5425" width="0.4064" layer="1"/>
+<wire x1="54.7116" y1="25.1206" x2="54.7116" y2="22.6822" width="0.8128" layer="1"/>
+<wire x1="54.7116" y1="22.6822" x2="54.61" y2="22.5425" width="0.4064" layer="1"/>
 <wire x1="54.7116" y1="27.1272" x2="54.6875" y2="27.33" width="0.4064" layer="1"/>
 <wire x1="29.5275" y1="45.1104" x2="16.6116" y2="45.1104" width="0.8128" layer="1"/>
@@
 <contactref element="D1" pad="A"/>
 <contactref element="PL1" pad="1"/>
-<wire x1="47.0916" y1="13.7668" x2="47.0916" y2="23.1648" width="0.8128" layer="1"/>
+<wire x1="47.0916" y1="13.7668" x2="47.0916" y2="22.5298" width="0.8128" layer="1"/>
 <wire x1="48.1584" y1="12.7" x2="47.0916" y2="13.7668" width="0.8128" layer="1"/>
-<wire x1="47.0916" y1="23.1648" x2="46.99" y2="22.5425" width="0.4064" layer="1"/>
+<wire x1="47.0916" y1="22.5298" x2="46.99" y2="22.5425" width="0.4064" layer="1"/>
 <wire x1="48.1584" y1="12.7" x2="48.26" y2="11.43" width="0.8128" layer="1"/>
 </signal>
