File: item_2022_Motherboard_04_V8.sch (EAGLE design)
At the start: 50 parts, among them IC1 MCP602SN, IC2 LD117AS33TR, IC4 MCP6S26, U1 ESP32-DEVKITC-32D, U2 ADS1256_BOARD, U3 SSD1306_128X64, X1 MSTBA4, X2 MSTBA4

Commit message: aggiunta su sch condizionamento coppie
Parts:
- removed JP1: (no value), pinhead:PINHD-1X8
- removed JP2: (no value), pinhead:PINHD-2X4
- added C12, C13, C15, C20, C29: 100nF, rcl_LargePads:C-EUC0805
- added C14: 10uF / 16V, rcl_LargePads:CPOL-EUC
- added C16, C17, C18, C19: 3.3uF/50V, rcl_LargePads:C-EUC0805
- added C21, C23, C25, C27: 2.2uF, rcl_LargePads:C-EUC0805
- added C22, C24, C26, C28: 1uF, rcl_LargePads:C-EUC0805
- added C30: 100nF, rcl:C-EUC0805
- added D2, D3, D4, D5: BZW06-10B, diode_LargePads:BZW04XXB
- added GND, GND36: TPTP18SQ, testpad:TPTP18SQ
- added IC3: MCP1525TO, MCP1525_MCP1541:MCP1525TO
- added IC5, IC6, IC9: MCP6004SO, MCP6002_MCP6004:MCP6004SO
- added IC7: MCP3204SL, MCP3204_MCP3208:MCP3204SL
- added IC8: LM336LP, linear:LM336LP
- added R10, R11: 6.8k, rcl_LargePads:R-EU_R0805
- added R12, R14, R22, R37, R39, R41, R43: 3.3k, rcl_LargePads:R-EU_R0805
- added R13, R19, R21, R23: 5.6k, rcl_LargePads:R-EU_R0805
- added R20: 3.3k, rcl_LargePads:R-EU_M0805
- added R24, R26, R28, R30: 2.7k, rcl_LargePads:R-EU_R0805
- added R25, R27, R29, R31: 82, rcl_LargePads:R-EU_R0805
- added R32, R33, R34, R35: 1.8k, rcl_LargePads:R-EU_R0805
- added R36, R38, R40, R42: 1.5k, rcl_LargePads:R-EU_R0805
- added R44: 2.7k, rcl:R-EU_R0805
- added R45, R46, R47, R48: 47, rcl:R-EU_R0805
- added R49: 10k, rcl:R-EU_R0805
- added TP13, TP7, TP8: TPTP16R, testpad:TPTP16R
- added TP14, TP15, TP16, TP17, TP18, TP19, TP20, TP21: TPTP14R, testpad:TPTP14R
Connections:
- removed net ADC_HALF_VREF: IC4.VREF, JP1.1, R16.1, R18.1, R2.1, R4.1, TP9.TP
- new net +2.5V: IC9D.-IN, IC9D.OUT, R32.1
- new net +3.3V_B: R49.2, U1.3V3
- new net ADC_HALF_VREF_A: IC4.VREF, IC9C.-IN, IC9C.OUT, R2.1, R4.1, TP13.TP, TP9.TP
- new net ADC_HALF_VREF_B: IC9A.-IN, IC9A.OUT, R16.1, R18.1
- new net ADC_VREF: IC7.VREF, IC9B.-IN, IC9B.OUT
- new net A_SPEED1: C25.2, IC6C.-IN, IC6C.OUT, IC7.CH2, TP20.TP
- new net A_SPEED2: C27.2, IC6D.-IN, IC6D.OUT, IC7.CH3, TP21.TP
- new net A_TORQUE1: C21.2, IC6A.-IN, IC6A.OUT, IC7.CH0, TP18.TP
- new net A_TORQUE2: C23.2, IC6B.-IN, IC6B.OUT, IC7.CH1, TP19.TP
- new net EN/!RESET!: C30.2, R49.1, U1.EN
- new net N$1: C15.1, IC9A.+IN, IC9C.+IN, R10.1, R11.2
- new net N$15: R12.1, R13.2
- new net N$16: R14.1, R19.2
- new net N$17: R20.1, R21.2
- new net N$18: R22.1, R23.2
- new net N$19: R24.2, R25.1
- new net N$20: C16.1, IC5A.+IN, R13.1, R24.1, R32.2, TP14.TP
- new net N$22: R26.2, R27.1
- new net N$23: R28.2, R29.1
- new net N$24: R30.2, R31.1
- new net N$25: C17.1, IC5B.+IN, R19.1, R26.1, R33.2, TP15.TP
- new net N$26: C18.1, IC5C.+IN, R21.1, R28.1, R34.2, TP16.TP
- new net N$27: C19.1, IC5D.+IN, R23.1, R30.1, R35.2, TP17.TP
- new net N$28: IC5A.-IN, IC5A.OUT, R36.1
- new net N$29: IC5B.-IN, IC5B.OUT, R38.1
- new net N$30: IC5C.-IN, IC5C.OUT, R40.1
- new net N$31: IC5D.-IN, IC5D.OUT, R42.1
- new net N$32: C21.1, R36.2, R37.1
- new net N$33: C22.1, IC6A.+IN, R37.2
- new net N$34: C23.1, R38.2, R39.1
- new net N$35: C24.1, IC6B.+IN, R39.2
- new net N$36: C25.1, R40.2, R41.1
- new net N$37: C26.1, IC6C.+IN, R41.2
- new net N$38: C27.1, R42.2, R43.1
- new net N$39: C28.1, IC6D.+IN, R43.2
- new net N$40: R48.1, U1.IO19
- new net N$41: IC7.CLK, R45.1
- new net N$42: IC7.DIN, R46.1
- new net N$43: IC7.!CS!/SHDN, R47.1
- new net VREF: C14.+, IC3.VOUT, IC8.C, IC9B.+IN, IC9D.+IN, R10.2, R44.1, TP8.TP
- net !CS_MCP3204!: now also R47.2; no longer JP1.5
- net +3V3: now also C29.1, IC7.VDD; no longer JP1.2
- net +5V: now also C12.1, C13.1, C20.1, IC3.VIN, IC5P.VDD, IC6P.VDD, IC9P.VDD, R44.2, TP7.TP; no longer JP1.3
- net GND: now also C12.2, C13.2, C14.-, C15.2, C16.2, C17.2, C18.2, C19.2, C20.2, C22.2, C24.2, C26.2, C28.2, C29.2, D2.2, D3.2, D4.2, D5.2, GND.TP, GND36.TP, IC3.VSS, IC5P.VSS, IC6P.VSS, IC7.AGND, IC7.DGND, IC8.A, IC9P.VSS, R11.1, R25.2, R27.2, R29.2, R31.2; no longer JP1.4
- net SPEED1+: now also D3.1, R20.2; no longer JP2.6
- net SPEED1-: no longer JP2.5
- net SPEED2+: now also D4.1, R22.2; no longer JP2.8
- net SPEED2-: no longer JP2.7
- net TORQUE1+: now also D5.1, R12.2; no longer JP2.2
- net TORQUE1-: no longer JP2.1
- net TORQUE2+: now also D2.1, R14.2; no longer JP2.4
- net TORQUE2-: no longer JP2.3
- net VSPI_MISO: now also IC7.DOUT, R48.2; no longer JP1.7, U1.IO19
- net VSPI_MOSI: now also R46.2; no longer JP1.8
- net VSPI_SCK: now also R45.2; no longer JP1.6
Other:
- note added: "Bidirezionale, 10.2V"
- note added: "Codice RS: 915-9312"
- note added: "Condensatori Poliestere"
- note added: "IC3 o IC8"
- note added: "Passa Basso, II ordine Taglio: 50Hz, Butterworth Guadagno x1"
- note added: "Poliestere"
- note added: "Sezione Vref e ADC Condizionamento coppie"
- note added: "Taglio: 49,46Hz"
- note removed: "Alla scheda piggy-back condizionamento torque/speed"

Commit message: aggiunta su brd cond coppie da sbrogliare
Connections:
- removed net SPEED1-: PL1.11
- removed net SPEED2-: PL1.13
- removed net TORQUE1-: PL1.7
- removed net TORQUE2-: PL1.9
- net +2.5V: now also R33.1, R34.1, R35.1
- net GND: now also C30.1, PL1.11, PL1.13, PL1.7, PL1.9
Changed lines of the file:
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@@
 </segment>
 <segment>
-<wire x1="101.6" y1="149.86" x2="106.68" y2="149.86" width="0.1524" layer="91"/>
+<wire x1="101.6" y1="149.86" x2="104.14" y2="149.86" width="0.1524" layer="91"/>
 <label x="101.6" y="149.86" size="1.27" layer="95" rot="R180" xref="yes"/>
 <pinref part="PL1" gate="G$1" pin="5"/>
+<pinref part="PL1" gate="G$1" pin="13"/>
+<wire x1="104.14" y1="149.86" x2="106.68" y2="149.86" width="0.1524" layer="91"/>
+<wire x1="106.68" y1="139.7" x2="104.14" y2="139.7" width="0.1524" layer="91"/>
+<wire x1="104.14" y1="139.7" x2="104.14" y2="142.24" width="0.1524" layer="91"/>
+<junction x="104.14" y="149.86"/>
+<pinref part="PL1" gate="G$1" pin="7"/>
+<wire x1="104.14" y1="142.24" x2="104.14" y2="144.78" width="0.1524" layer="91"/>
+<wire x1="104.14" y1="144.78" x2="104.14" y2="147.32" width="0.1524" layer="91"/>
+<wire x1="104.14" y1="147.32" x2="104.14" y2="149.86" width="0.1524" layer="91"/>
+<wire x1="106.68" y1="147.32" x2="104.14" y2="147.32" width="0.1524" layer="91"/>
+<junction x="104.14" y="147.32"/>
+<pinref part="PL1" gate="G$1" pin="9"/>
+<wire x1="106.68" y1="144.78" x2="104.14" y2="144.78" width="0.1524" layer="91"/>
+<junction x="104.14" y="144.78"/>
+<pinref part="PL1" gate="G$1" pin="11"/>
+<wire x1="106.68" y1="142.24" x2="104.14" y2="142.24" width="0.1524" layer="91"/>
+<junction x="104.14" y="142.24"/>
 </segment>
 <segment>
@@
 <segment>
 <pinref part="GND34" gate="1" pin="GND"/>
+<pinref part="C30" gate="G$1" pin="1"/>
 <wire x1="200.66" y1="83.82" x2="200.66" y2="88.9" width="0.1524" layer="91"/>
 </segment>
@@
 </segment>
 </net>
-<net name="TORQUE1-" class="3">
-<segment>
-<wire x1="101.6" y1="147.32" x2="106.68" y2="147.32" width="0.1524" layer="91"/>
-<label x="101.6" y="147.32" size="1.27" layer="95" rot="R180" xref="yes"/>
-<pinref part="PL1" gate="G$1" pin="7"/>
-</segment>
-</net>
-<net name="TORQUE2-" class="3">
-<segment>
-<wire x1="101.6" y1="144.78" x2="106.68" y2="144.78" width="0.1524" layer="91"/>
-<label x="101.6" y="144.78" size="1.27" layer="95" rot="R180" xref="yes"/>
-<pinref part="PL1" gate="G$1" pin="9"/>
-</segment>
-</net>
 <net name="SPEED1+" class="3">
 <segment>
@@
 <pinref part="PL1" gate="G$1" pin="12"/>
 <label x="127" y="142.24" size="1.27" layer="95" xref="yes"/>
-</segment>
-</net>
-<net name="SPEED1-" class="3">
-<segment>
-<wire x1="101.6" y1="142.24" x2="106.68" y2="142.24" width="0.1524" layer="91"/>
-<label x="101.6" y="142.24" size="1.27" layer="95" rot="R180" xref="yes"/>
-<pinref part="PL1" gate="G$1" pin="11"/>
-</segment>
-</net>
-<net name="SPEED2-" class="3">
-<segment>
-<wire x1="101.6" y1="139.7" x2="106.68" y2="139.7" width="0.1524" layer="91"/>
-<label x="101.6" y="139.7" size="1.27" layer="95" rot="R180" xref="yes"/>
-<pinref part="PL1" gate="G$1" pin="13"/>
 </segment>
 </net>
@@
 <segment>
 <pinref part="R32" gate="G$1" pin="1"/>
+<wire x1="116.84" y1="218.44" x2="116.84" y2="215.9" width="0.1524" layer="91"/>
+<label x="116.84" y="218.44" size="1.27" layer="95" rot="R90" xref="yes"/>
+<pinref part="R33" gate="G$1" pin="1"/>
 <wire x1="116.84" y1="215.9" x2="116.84" y2="213.36" width="0.1524" layer="91"/>
-<label x="116.84" y="215.9" size="1.27" layer="95" rot="R90" xref="yes"/>
-</segment>
-<segment>
-<wire x1="134.62" y1="215.9" x2="134.62" y2="213.36" width="0.1524" layer="91"/>
-<label x="134.62" y="215.9" size="1.27" layer="95" rot="R90" xref="yes"/>
-</segment>
-<segment>
-<wire x1="152.4" y1="215.9" x2="152.4" y2="213.36" width="0.1524" layer="91"/>
-<label x="152.4" y="215.9" size="1.27" layer="95" rot="R90" xref="yes"/>
-</segment>
-<segment>
-<wire x1="170.18" y1="215.9" x2="170.18" y2="213.36" width="0.1524" layer="91"/>
-<label x="170.18" y="215.9" size="1.27" layer="95" rot="R90" xref="yes"/>
-</segment>
-</net>
+<wire x1="134.62" y1="213.36" x2="134.62" y2="215.9" width="0.1524" layer="91"/>
+<wire x1="134.62" y1="215.9" x2="116.84" y2="215.9" width="0.1524" layer="91"/>
+<junction x="116.84" y="215.9"/>
+<pinref part="R34" gate="G$1" pin="1"/>
+<wire x1="152.4" y1="213.36" x2="152.4" y2="215.9" width="0.1524" layer="91"/>
+<wire x1="152.4" y1="215.9" x2="134.62" y2="215.9" width="0.1524" layer="91"/>
+<junction x="134.62" y="215.9"/>
+<pinref part="R35" gate="G$1" pin="1"/>
+<wire x1="170.18" y1="213.36" x2="170.18" y2="215.9" width="0.1524" layer="91"/>
+<wire x1="170.18" y1="215.9" x2="152.4" y2="215.9" width="0.1524" layer="91"/>
+<junction x="152.4" y="215.9"/>
+</segment>
+</net>

Commit message: changed PGA inputs
Connections:
- net GND: now also IC4.CH0, IC4.CH2, IC4.CH4, IC4.CH5
- net N$14: now also IC4.CH3; no longer IC4.CH1
- net N$4: now also IC4.CH1; no longer IC4.CH0
Other:
- moved on the sheet: C1, C2, R1, R2, R3, R4, TP1, TP2, TP5, TP6, X1-1, X1-2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

Commit message: routing with corrected pads
Other:
- note added: "Lista Tesp Points: TP1 - ingresso Accel_0 TP2 - Accel_0 con bias TP3 - uscita PGA Accel_0/1 TP4 - uscita LPF Accel_0/AIN0+ TP5 - ingresso Accel_1 TP6 - Accel_1 con bias TP7 - +5V TP8 - VREF +2.5V TP9 - ADC_HALF_VREF TP10 - +3V3 TP11 - +5V TP12 - GND TP13 - ADC_HALF_VREF_A TP14 - TORQUE1_NORM TP15 - TORQUE2_NORM TP16 - SPEED1_NORM TP17 - SPEED2_NORM TP18 - A_TORQUE1 TP19 - A_TORQUE2 TP20 - A_SPEED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"
- note removed: "Lista Tesp Points: TP1 - ingresso Accel_0 TP2 - Accel_0 con bias TP3 - uscita PGA Accel_0/1 TP4 - uscita LPF Accel_0/AIN0+ TP5 - ingresso Accel_1 TP6 - Accel_1 con bias TP9 - ADC_HALF_VREF TP10 - +3V3 TP11 - +5V TP12 - GND"
Changed lines of the file:
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@@
 Condizionamento coppie</text>
 <text x="346.71" y="20.32" size="2.54" layer="97">ISIS Bassa Friulana</text>
-<text x="289.56" y="33.02" size="2.1844" layer="97">Lista Tesp Points:
+<text x="332.74" y="33.02" size="2.1844" layer="97">Lista Tesp Points:
 TP1 - ingresso Accel_0
 TP2 - Accel_0 con bias
@@
 TP5 - ingresso Accel_1
 TP6 - Accel_1 con bias
+TP7 - +5V
+TP8 - VREF +2.5V
 TP9 - ADC_HALF_VREF
 TP10 - +3V3
 TP11 - +5V
 TP12 - GND
-</text>
+TP13 - ADC_HALF_VREF_A
+TP14 - TORQUE1_NORM
+TP15 - TORQUE2_NORM
+TP16 - SPEED1_NORM
+TP17 - SPEED2_NORM
+TP18 - A_TORQUE1
+TP19 - A_TORQUE2
+TP20 - A_SPEED1
+TP21 - A_SPEED2</text>
 <text x="20.32" y="86.36" size="1.778" layer="97">Segnali di PL1 verso scheda front-end:
 1. Ext.Supply +5V

Commit message: cambio package elettrolitici smd
Parts:
- added C31: 220uF/16V, rcl@1:CPOL-EUE3.5-10
- C14: value 10uF / 16V -> 10uF/16V; device rcl_LargePads:CPOL-EUC -> rcl@1:CPOL-EUE2.5-6
- C4: device rcl@1:CPOL-EUE3.5-8 -> rcl@1:CPOL-EUE2.5-6
Connections:
- net +5V: now also C31.+
- net GND: now also C31.-
Changed lines of the file:
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@@
 <setting verticaltext="up"/>
 </settings>
-<grid distance="0.1" unitdist="inch" unit="inch" style="lines" multiple="1" display="no" altdistance="0.01" altunitdist="inch" altunit="inch"/>
+<grid distance="0.1" unitdist="inch" unit="inch" style="lines" multiple="1" display="yes" altdistance="0.01" altunitdist="inch" altunit="inch"/>
 <layers>
-<layer number="1" name="Top" color="4" fill="1" visible="no" active="no"/>
-<layer number="2" name="Route2" color="1" fill="3" visible="no" active="no"/>
-<layer number="3" name="Route3" color="4" fill="3" visible="no" active="no"/>
-<layer number="14" name="Route14" color="1" fill="6" visible="no" active="no"/>
-<layer number="15" name="Route15" color="4" fill="6" visible="no" active="no"/>
-<layer number="16" name="Bottom" color="1" fill="1" visible="no" active="no"/>
-<layer number="17" name="Pads" color="2" fill="1" visible="no" active="no"/>
-<layer number="18" name="Vias" color="2" fill="1" visible="no" active="no"/>
-<layer number="19" name="Unrouted" color="6" fill="1" visible="no" active="no"/>
-<layer number="20" name="Dimension" color="15" fill="1" visible="no" active="no"/>
-<layer number="21" name="tPlace" color="7" fill="1" visible="no" active="no"/>
-<layer number="22" name="bPlace" color="7" fill="1" visible="no" active="no"/>
-<layer number="23" name="tOrigins" color="15" fill="1" visible="no" active="no"/>
-<layer number="24" name="bOrigins" color="15" fill="1" visible="no" active="no"/>
-<layer number="25" name="tNames" color="7" fill="1" visible="no" active="no"/>
-<layer number="26" name="bNames" color="7" fill="1" visible="no" active="no"/>
-<layer number="27" name="tValues" color="7" fill="1" visible="no" active="no"/>
-<layer number="28" name="bValues" color="7" fill="1" visible="no" active="no"/>
+<layer number="1" name="Top" color="4" fill="1" visible="yes" active="no"/>
+<layer number="2" name="Route2" color="1" fill="3" visible="yes" active="no"/>
+<layer number="3" name="Route3" color="4" fill="3" visible="yes" active="no"/>
+<layer number="14" name="Route14" color="1" fill="6" visible="yes" active="no"/>
+<layer number="15" name="Route15" color="4" fill="6" visible="yes" active="no"/>
+<layer number="16" name="Bottom" color="1" fill="1" visible="yes" active="no"/>
+<layer number="17" name="Pads" color="2" fill="1" visible="yes" active="no"/>
+<layer number="18" name="Vias" color="2" fill="1" visible="yes" active="no"/>
+<layer number="19" name="Unrouted" color="6" fill="1" visible="yes" active="no"/>
+<layer number="20" name="Dimension" color="15" fill="1" visible="yes" active="no"/>
+<layer number="21" name="tPlace" color="7" fill="1" visible="yes" active="no"/>
+<layer number="22" name="bPlace" color="7" fill="1" visible="yes" active="no"/>
+<layer number="23" name="tOrigins" color="15" fill="1" visible="yes" active="no"/>
+<layer number="24" name="bOrigins" color="15" fill="1" visible="yes" active="no"/>
+<layer number="25" name="tNames" color="7" fill="1" visible="yes" active="no"/>
+<layer number="26" name="bNames" color="7" fill="1" visible="yes" active="no"/>
+<layer number="27" name="tValues" color="7" fill="1" visible="yes" active="no"/>
+<layer number="28" name="bValues" color="7" fill="1" visible="yes" active="no"/>
 <layer number="29" name="tStop" color="7" fill="3" visible="no" active="no"/>
 <layer number="30" name="bStop" color="7" fill="6" visible="no" active="no"/>
@@
 <layer number="35" name="tGlue" color="7" fill="4" visible="no" active="no"/>
 <layer number="36" name="bGlue" color="7" fill="5" visible="no" active="no"/>
-<layer number="37" name="tTest" color="7" fill="1" visible="no" active="no"/>
-<layer number="38" name="bTest" color="7" fill="1" visible="no" active="no"/>
+<layer number="37" name="tTest" color="7" fill="1" visible="yes" active="no"/>
+<layer number="38" name="bTest" color="7" fill="1" visible="yes" active="no"/>
 <layer number="39" name="tKeepout" color="4" fill="11" visible="no" active="no"/>
 <layer number="40" name="bKeepout" color="1" fill="11" visible="no" active="no"/>
@@
 <layer number="44" name="Drills" color="7" fill="1" visible="no" active="no"/>
 <layer number="45" name="Holes" color="7" fill="1" visible="no" active="no"/>
-<layer number="46" name="Milling" color="3" fill="1" visible="no" active="no"/>
-<layer number="47" name="Measures" color="7" fill="1" visible="no" active="no"/>
-<layer number="48" name="Document" color="7" fill="1" visible="no" active="no"/>
-<layer number="49" name="Reference" color="7" fill="1" visible="no" active="no"/>
-<layer number="51" name="tDocu" color="7" fill="1" visible="no" active="no"/>
-<layer number="52" name="bDocu" color="7" fill="1" visible="no" active="no"/>
+<layer number="46" name="Milling" color="3" fill="1" visible="yes" active="no"/>
+<layer number="47" name="Measures" color="7" fill="1" visible="yes" active="no"/>
+<layer number="48" name="Document" color="7" fill="1" visible="yes" active="no"/>
+<layer number="49" name="Reference" color="7" fill="1" visible="yes" active="no"/>
+<layer number="51" name="tDocu" color="7" fill="1" visible="yes" active="no"/>
+<layer number="52" name="bDocu" color="7" fill="1" visible="yes" active="no"/>
 <layer number="88" name="SimResults" color="9" fill="1" visible="yes" active="yes"/>
 <layer number="89" name="SimProbes" color="9" fill="1" visible="yes" active="yes"/>
@@
 <part name="JP4" library="pinhead" deviceset="PINHD-1X15" device=""/>
 <part name="GND16" library="supply1" deviceset="GND" device=""/>
-<part name="C4" library="rcl@1" deviceset="CPOL-EU" device="E3.5-8" value="10uF/16V"/>
+<part name="C4" library="rcl@1" deviceset="CPOL-EU" device="E2.5-6" value="10uF/16V"/>
 <part name="IC1" library="linear" deviceset="MCP602" device="SN"/>
 <part name="GND17" library="supply1" deviceset="GND" device=""/>
@@
 <part name="GND20" library="supply1" deviceset="GND" device=""/>
 <part name="P+6" library="supply1" deviceset="+5V" device=""/>
-<part name="C14" library="rcl_LargePads" deviceset="CPOL-EU" device="C" value="10uF / 16V"/>
 <part name="R10" library="rcl_LargePads" deviceset="R-EU_" device="R0805" value="6.8k"/>
 <part name="R11" library="rcl_LargePads" deviceset="R-EU_" device="R0805" value="6.8k"/>
@@
 <part name="C30" library="rcl" deviceset="C-EU" device="C0805" value="100nF"/>
 <part name="GND34" library="supply1" deviceset="GND" device=""/>
+<part name="C14" library="rcl@1" deviceset="CPOL-EU" device="E2.5-6" value="10uF/16V"/>
+<part name="C31" library="rcl@1" deviceset="CPOL-EU" device="E3.5-10" value="220uF/16V"/>
 </parts>
 <sheets>
@@
 <attribute name="VALUE" x="198.12" y="78.74" size="1.778" layer="96"/>
 </instance>
+<instance part="C31" gate="G$1" x="88.9" y="33.02" smashed="yes">
+<attribute name="NAME" x="90.043" y="33.5026" size="1.778" layer="95"/>
+<attribute name="VALUE" x="90.043" y="28.4226" size="1.778" layer="96"/>
+</instance>
 </instances>
 <busses>
@@
 <pinref part="IC2" gate="G$1" pin="ADJ"/>
 <wire x1="106.68" y1="33.02" x2="106.68" y2="22.86" width="0.1524" layer="91"/>
-<wire x1="106.68" y1="22.86" x2="71.12" y2="22.86" width="0.1524" layer="91"/>
+<wire x1="106.68" y1="22.86" x2="88.9" y2="22.86" width="0.1524" layer="91"/>
 <junction x="71.12" y="22.86"/>
+<wire x1="88.9" y1="22.86" x2="71.12" y2="22.86" width="0.1524" layer="91"/>
 <wire x1="129.54" y1="27.94" x2="129.54" y2="22.86" width="0.1524" layer="91"/>
 <wire x1="129.54" y1="22.86" x2="106.68" y2="22.86" width="0.1524" layer="91"/>
@@
 <wire x1="162.56" y1="25.4" x2="162.56" y2="22.86" width="0.1524" layer="91"/>
 <pinref part="C4" gate="G$1" pin="-"/>
+<pinref part="C31" gate="G$1" pin="-"/>
+<wire x1="88.9" y1="27.94" x2="88.9" y2="22.86" width="0.1524" layer="91"/>
+<junction x="88.9" y="22.86"/>
 </segment>
 <segment>
@@
 <wire x1="88.9" y1="43.18" x2="88.9" y2="40.64" width="0.1524" layer="91"/>
 <junction x="88.9" y="40.64"/>
+<pinref part="C31" gate="G$1" pin="+"/>
+<wire x1="88.9" y1="35.56" x2="88.9" y2="40.64" width="0.1524" layer="91"/>
 </segment>
 </net>
@@
 <attribute name="VALUE" x="180.34" y="43.18" size="1.4224" layer="96" rot="R90"/>
 </instance>
-<instance part="C14" gate="G$1" x="66.04" y="53.34" smashed="yes">
-<attribute name="NAME" x="67.183" y="53.8226" size="1.778" layer="95"/>
-<attribute name="VALUE" x="67.183" y="48.7426" size="1.778" layer="96"/>
-</instance>
 <instance part="R10" gate="G$1" x="86.36" y="48.26" smashed="yes" rot="R90">
 <attribute name="NAME" x="84.8614" y="44.45" size="1.778" layer="95" rot="R90"/>
@@
 <instance part="R46" gate="G$1" x="325.12" y="58.42"/>
 <instance part="R47" gate="G$1" x="314.96" y="55.88"/>
+<instance part="C14" gate="G$1" x="66.04" y="53.34" smashed="yes">
+<attribute name="NAME" x="67.183" y="53.8226" size="1.778" layer="95"/>
+<attribute name="VALUE" x="67.183" y="48.7426" size="1.778" layer="96"/>
+</instance>
 </instances>
 <busses>
@@
 <pinref part="IC3" gate="G$1" pin="VOUT"/>
 <wire x1="58.42" y1="60.96" x2="66.04" y2="60.96" width="0.1524" layer="91"/>
-<pinref part="C14" gate="G$1" pin="+"/>
 <wire x1="66.04" y1="60.96" x2="86.36" y2="60.96" width="0.1524" layer="91"/>
-<wire x1="86.36" y1="60.96" x2="86.36" y2="81.28" width="0.1524" layer="91"/>
 <wire x1="86.36" y1="81.28" x2="93.98" y2="81.28" width="0.1524" layer="91"/>
-<wire x1="66.04" y1="55.88" x2="66.04" y2="60.96" width="0.1524" layer="91"/>
 <junction x="66.04" y="60.96"/>
 <pinref part="R10" gate="G$1" pin="2"/>
@@
 <junction x="86.36" y="101.6"/>
 <junction x="86.36" y="81.28"/>
-</segment>
-</net>
+<pinref part="C14" gate="G$1" pin="+"/>
+<wire x1="66.04" y1="55.88" x2="66.04" y2="60.96" width="0.1524" layer="91"/>
+</segment>
+</net>
