File: item_2022_Motherboard_04_V8.sch (EAGLE design)
At the start: 123 parts, among them IC1 MCP602SN, IC2 LD117AS33TR, IC3 MCP1525TO, IC4 MCP6S28DIL, IC5 MCP6004SO, IC6 MCP6004SO, IC7 MCP3204SL, IC8 LM336LP, IC9 MCP6004SO, U1 ESP32-DEVKITC-32D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

Commit message: corretto diametro SSD1306 e RTD
Other:
- note added: "Sezione logica e ADC Condizionamento RTD"
- note removed: "Sezione logica e ADC Condizionamento coppie"
Changed lines of the file:
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@@
 <setting verticaltext="up"/>
 </settings>
-<grid distance="0.05" unitdist="inch" unit="inch" style="lines" multiple="1" display="yes" altdistance="0.01" altunitdist="inch" altunit="inch"/>
+<grid distance="0.1" unitdist="inch" unit="inch" style="lines" multiple="1" display="no" altdistance="0.01" altunitdist="inch" altunit="inch"/>
 <layers>
 <layer number="1" name="Top" color="4" fill="1" visible="no" active="no"/>
@@
 <plain>
 <text x="292.1" y="12.7" size="2.54" layer="97">Sezione logica e ADC
-Condizionamento coppie</text>
+Condizionamento RTD</text>
 <text x="346.71" y="20.32" size="2.54" layer="97">ISIS Bassa Friulana</text>
 <text x="332.74" y="33.02" size="2.1844" layer="97">Lista Tesp Points:

Commit message: Corretto pinout MCP1525
Changed lines of the file:
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@@
 <attribute name="NAME" x="118.11" y="133.858" size="1.778" layer="95" rot="R180"/>
 </instance>
-<instance part="R48" gate="G$1" x="99.06" y="220.98"/>
-<instance part="R49" gate="G$1" x="200.66" y="106.68" rot="R90"/>
-<instance part="C30" gate="G$1" x="200.66" y="91.44" rot="R180"/>
+<instance part="R48" gate="G$1" x="99.06" y="220.98" smashed="yes">
+<attribute name="NAME" x="95.25" y="222.4786" size="1.778" layer="95"/>
+<attribute name="VALUE" x="95.25" y="217.678" size="1.778" layer="96"/>
+</instance>
+<instance part="R49" gate="G$1" x="200.66" y="106.68" smashed="yes" rot="R90">
+<attribute name="NAME" x="199.1614" y="102.87" size="1.778" layer="95" rot="R90"/>
+<attribute name="VALUE" x="203.962" y="102.87" size="1.778" layer="96" rot="R90"/>
+</instance>
+<instance part="C30" gate="G$1" x="200.66" y="91.44" smashed="yes" rot="R180">
+<attribute name="NAME" x="199.136" y="91.059" size="1.778" layer="95" rot="R180"/>
+<attribute name="VALUE" x="199.136" y="96.139" size="1.778" layer="96" rot="R180"/>
+</instance>
 <instance part="GND34" gate="1" x="200.66" y="81.28" smashed="yes">
 <attribute name="VALUE" x="198.12" y="78.74" size="1.778" layer="96"/>
@@
 <attribute name="VALUE" x="90.043" y="28.4226" size="1.778" layer="96"/>
 </instance>
-<instance part="U3" gate="G$1" x="213.36" y="231.14"/>
+<instance part="U3" gate="G$1" x="213.36" y="231.14" smashed="yes">
+<attribute name="NAME" x="205.74" y="240.03" size="1.27" layer="95"/>
+<attribute name="VALUE" x="205.74" y="223.52" size="1.27" layer="95"/>
+</instance>
 </instances>
 <busses>
@@
 <attribute name="VALUE" x="172.72" y="228.6" size="1.4224" layer="96" rot="R90"/>
 </instance>
-<instance part="IC4" gate="G$1" x="175.26" y="182.88"/>
+<instance part="IC4" gate="G$1" x="175.26" y="182.88" smashed="yes">
+<attribute name="NAME" x="165.1" y="207.01" size="1.27" layer="95"/>
+<attribute name="VALUE" x="165.1" y="165.1" size="1.27" layer="96"/>
+</instance>
 </instances>
 <busses>
@@
 <attribute name="TP_SIGNAL_NAME" x="293.37" y="125.73" size="1.778" layer="97"/>
 </instance>
-<instance part="R45" gate="G$1" x="314.96" y="63.5"/>
-<instance part="R46" gate="G$1" x="325.12" y="58.42"/>
-<instance part="R47" gate="G$1" x="314.96" y="55.88"/>
+<instance part="R45" gate="G$1" x="314.96" y="63.5" smashed="yes">
+<attribute name="NAME" x="311.15" y="64.9986" size="1.778" layer="95"/>
+<attribute name="VALUE" x="311.15" y="60.198" size="1.778" layer="96"/>
+</instance>
+<instance part="R46" gate="G$1" x="325.12" y="58.42" smashed="yes">
+<attribute name="NAME" x="321.31" y="59.9186" size="1.778" layer="95"/>
+<attribute name="VALUE" x="321.31" y="55.118" size="1.778" layer="96"/>
+</instance>
+<instance part="R47" gate="G$1" x="314.96" y="55.88" smashed="yes">
+<attribute name="NAME" x="311.15" y="57.3786" size="1.778" layer="95"/>
+<attribute name="VALUE" x="311.15" y="52.578" size="1.778" layer="96"/>
+</instance>
 <instance part="C14" gate="G$1" x="66.04" y="53.34" smashed="yes">
 <attribute name="NAME" x="67.183" y="53.8226" size="1.778" layer="95"/>
@@
 <pinref part="GND18" gate="1" pin="GND"/>
 <wire x1="66.04" y1="43.18" x2="48.26" y2="43.18" width="0.1524" layer="91"/>
-<pinref part="IC3" gate="G$1" pin="VSS"/>
-<wire x1="48.26" y1="50.8" x2="48.26" y2="43.18" width="0.1524" layer="91"/>
 <junction x="48.26" y="43.18"/>
 <pinref part="C12" gate="G$1" pin="2"/>
@@
 <pinref part="C14" gate="G$1" pin="-"/>
 <wire x1="66.04" y1="48.26" x2="66.04" y2="43.18" width="0.1524" layer="91"/>
+<pinref part="IC3" gate="G$1" pin="VSS"/>
+<wire x1="48.26" y1="50.8" x2="48.26" y2="43.18" width="0.1524" layer="91"/>
 </segment>
 <segment>
@@
 <net name="+5V" class="4">
 <segment>
-<wire x1="35.56" y1="66.04" x2="35.56" y2="60.96" width="0.1524" layer="91"/>
-<pinref part="IC3" gate="G$1" pin="VIN"/>
-<wire x1="35.56" y1="60.96" x2="38.1" y2="60.96" width="0.1524" layer="91"/>
 <pinref part="P+4" gate="1" pin="+5V"/>
 <pinref part="C12" gate="G$1" pin="1"/>
 <wire x1="35.56" y1="53.34" x2="35.56" y2="60.96" width="0.1524" layer="91"/>
+<pinref part="IC3" gate="G$1" pin="VIN"/>
+<wire x1="35.56" y1="60.96" x2="35.56" y2="66.04" width="0.1524" layer="91"/>
+<wire x1="38.1" y1="60.96" x2="35.56" y2="60.96" width="0.1524" layer="91"/>
 <junction x="35.56" y="60.96"/>
 </segment>
@@
 <wire x1="66.04" y1="86.36" x2="66.04" y2="88.9" width="0.1524" layer="91"/>
 <junction x="66.04" y="86.36"/>
-<pinref part="IC3" gate="G$1" pin="VOUT"/>
-<wire x1="58.42" y1="60.96" x2="66.04" y2="60.96" width="0.1524" layer="91"/>
 <wire x1="66.04" y1="60.96" x2="86.36" y2="60.96" width="0.1524" layer="91"/>
 <wire x1="86.36" y1="81.28" x2="93.98" y2="81.28" width="0.1524" layer="91"/>
@@
 <pinref part="C14" gate="G$1" pin="+"/>
 <wire x1="66.04" y1="55.88" x2="66.04" y2="60.96" width="0.1524" layer="91"/>
-</segment>
-</net>
+<pinref part="IC3" gate="G$1" pin="VOUT"/>
+<wire x1="58.42" y1="60.96" x2="66.04" y2="60.96" width="0.1524" layer="91"/>
+</segment>
+</net>
