File: item_2022_Frontend_02_V7.brd (EAGLE design)
At the start: 160 x 100 mm, 29 parts, among them K1 351, U3 SSD1306_128X64, X1 MSTBA2, X10 MSTBA2, X11 MSTBA2, X12 MSTBA2, X13 MSTBA2, X14 MSTBA2, X15 MSTBA2, X2 MSTBA2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

Commit message: spostati BZW su Frontend da motherboard
Parts:
- added D2, D3, D4, D5: BZW06-10B, diode_LargePads:F126Z12
Connections:
- removed net SPEED1-: PL1.11, X4.2
- removed net SPEED2-: PL1.13, X5.2
- removed net TORQUE1-: PL1.7, X2.2
- removed net TORQUE2-: PL1.9, X3.2
- net GND: now also D2.C, D3.C, D4.C, D5.C, PL1.11, PL1.13, PL1.7, PL1.9, X2.2, X3.2, X4.2, X5.2
- net SPEED1+: now also D3.A
- net SPEED2+: now also D4.A
- net TORQUE1+: now also D5.A
- net TORQUE2+: now also D2.A
Routing:
- net SPEED2-: track 86.5 -> 0.00 mm
- net TORQUE1-: track 81.7 -> 0.00 mm
- net SPEED1-: track 81.7 -> 0.00 mm
- net TORQUE2-: track 77.5 -> 0.00 mm
- net SPEED1+: track 130.7 -> 148.4 mm
- net SPEED2+: track 102.8 -> 120.3 mm
- net TORQUE1+: track 95.9 -> 101.7 mm
- net TORQUE2+: track 111.2 -> 114.8 mm
Changed lines of the file:
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@@
 <attribute name="MPN" value="" x="39.37" y="11.43" size="1.778" layer="27" rot="R180" display="off"/>
+</element>
+<element name="D2" library="diode_LargePads" package="F126Z12" value="BZW06-10B" x="46.355" y="72.39">
+<attribute name="POPULARITY" value="0" x="46.355" y="72.39" size="1.778" layer="27" display="off"/>
+</element>
+<element name="D3" library="diode_LargePads" package="F126Z12" value="BZW06-10B" x="24.13" y="72.39">
+<attribute name="POPULARITY" value="0" x="24.13" y="72.39" size="1.778" layer="27" display="off"/>
+</element>
+<element name="D4" library="diode_LargePads" package="F126Z12" value="BZW06-10B" x="24.13" y="66.04">
+<attribute name="POPULARITY" value="0" x="24.13" y="66.04" size="1.778" layer="27" display="off"/>
+</element>
+<element name="D5" library="diode_LargePads" package="F126Z12" value="BZW06-10B" x="46.355" y="66.04">
+<attribute name="POPULARITY" value="0" x="46.355" y="66.04" size="1.778" layer="27" display="off"/>
 </element>
 </elements>
@@
 <via x="85.09" y="12.065" extent="1-16" drill="0.6"/>
 <via x="92.71" y="17.78" extent="1-16" drill="0.6"/>
-<wire x1="85.09" y1="12.065" x2="92.71" y2="17.78" width="0" layer="19" extent="1-1"/>
+<contactref element="X5" pad="2"/>
+<contactref element="X4" pad="2"/>
+<contactref element="X3" pad="2"/>
+<contactref element="X2" pad="2"/>
+<contactref element="D5" pad="C"/>
+<contactref element="D4" pad="C"/>
+<contactref element="D3" pad="C"/>
+<contactref element="D2" pad="C"/>
+<contactref element="PL1" pad="7"/>
+<contactref element="PL1" pad="9"/>
+<contactref element="PL1" pad="11"/>
+<contactref element="PL1" pad="13"/>
 </signal>
 <signal name="I2C_SCL">
@@
 <wire x1="49.9872" y1="13.208" x2="49.9872" y2="9.5504" width="0.889" layer="1"/>
 <wire x1="46.9392" y1="16.256" x2="49.9872" y2="13.208" width="0.889" layer="1"/>
-<wire x1="46.9392" y1="81.0768" x2="46.9392" y2="16.256" width="0.889" layer="1"/>
+<wire x1="46.9392" y1="81.0768" x2="46.9392" y2="66.04" width="0.889" layer="1"/>
+<wire x1="46.9392" y1="66.04" x2="46.9392" y2="16.256" width="0.889" layer="1"/>
 <wire x1="55.88" y1="90.0176" x2="46.9392" y2="81.0768" width="0.889" layer="1"/>
 <wire x1="43.0784" y1="10.16" x2="43.18" y2="10.16" width="0.889" layer="1"/>
 <wire x1="55.88" y1="90.0176" x2="55.88" y2="90.17" width="0.889" layer="1"/>
+<contactref element="D5" pad="A"/>
+<wire x1="52.705" y1="66.04" x2="46.9392" y2="66.04" width="0.889" layer="1"/>
 </signal>
 <signal name="TORQUE2+" class="2">
@@
 <wire x1="50.8" y1="13.8176" x2="50.8" y2="10.3632" width="0.889" layer="16"/>
 <wire x1="56.2864" y1="19.304" x2="50.8" y2="13.8176" width="0.889" layer="16"/>
-<wire x1="56.2864" y1="85.9536" x2="56.2864" y2="19.304" width="0.889" layer="16"/>
+<wire x1="56.2864" y1="85.9536" x2="56.2864" y2="72.39" width="0.889" layer="16"/>
+<wire x1="56.2864" y1="72.39" x2="56.2864" y2="19.304" width="0.889" layer="16"/>
 <wire x1="52.832" y1="89.408" x2="56.2864" y2="85.9536" width="0.889" layer="16"/>
 <wire x1="52.832" y1="92.0496" x2="52.832" y2="89.408" width="0.889" layer="16"/>
@@
 <wire x1="43.2816" y1="90.2208" x2="43.18" y2="90.17" width="0.889" layer="16"/>
 <via x="42.8752" y="6.2992" extent="1-16" drill="0.6096"/>
-</signal>
-<signal name="TORQUE1-" class="2">
-<contactref element="X2" pad="2"/>
-<contactref element="PL1" pad="7"/>
-<wire x1="40.64" y1="79.8576" x2="40.64" y2="12.7" width="0.889" layer="16"/>
-<wire x1="50.8" y1="90.0176" x2="40.64" y2="79.8576" width="0.889" layer="16"/>
-<wire x1="50.8" y1="90.0176" x2="50.8" y2="90.17" width="0.889" layer="16"/>
-</signal>
-<signal name="TORQUE2-" class="2">
-<contactref element="X3" pad="2"/>
-<contactref element="PL1" pad="9"/>
-<wire x1="38.2016" y1="90.0176" x2="38.2016" y2="12.8016" width="0.889" layer="16"/>
-<wire x1="38.2016" y1="12.8016" x2="38.1" y2="12.7" width="0.889" layer="16"/>
-<wire x1="38.2016" y1="90.0176" x2="38.1" y2="90.17" width="0.889" layer="16"/>
+<contactref element="D2" pad="A"/>
+<wire x1="52.705" y1="72.39" x2="56.2864" y2="72.39" width="0.889" layer="16"/>
 </signal>
 <signal name="SPEED1+" class="2">
@@
 <wire x1="37.9984" y1="10.16" x2="38.1" y2="10.16" width="0.889" layer="1"/>
 <wire x1="30.48" y1="90.2208" x2="30.48" y2="90.17" width="0.889" layer="1"/>
+<contactref element="D3" pad="A"/>
+<wire x1="30.48" y1="72.39" x2="30.48" y2="90.17" width="0.889" layer="1"/>
 </signal>
 <signal name="SPEED2+" class="2">
@@
 <wire x1="24.9936" y1="6.096" x2="32.1056" y2="6.096" width="0.889" layer="1"/>
 <wire x1="14.0208" y1="17.0688" x2="24.9936" y2="6.096" width="0.889" layer="1"/>
-<wire x1="14.0208" y1="86.36" x2="14.0208" y2="17.0688" width="0.889" layer="1"/>
+<wire x1="14.0208" y1="86.36" x2="14.0208" y2="68.58" width="0.889" layer="1"/>
+<wire x1="14.0208" y1="68.58" x2="14.0208" y2="17.0688" width="0.889" layer="1"/>
 <wire x1="17.6784" y1="90.0176" x2="14.0208" y2="86.36" width="0.889" layer="1"/>
 <wire x1="17.6784" y1="90.0176" x2="17.78" y2="90.17" width="0.889" layer="1"/>
-</signal>
-<signal name="SPEED1-" class="2">
-<contactref element="X4" pad="2"/>
-<contactref element="PL1" pad="11"/>
-<wire x1="35.56" y1="79.8576" x2="35.56" y2="12.7" width="0.889" layer="16"/>
-<wire x1="25.4" y1="90.0176" x2="35.56" y2="79.8576" width="0.889" layer="16"/>
-<wire x1="25.4" y1="90.0176" x2="25.4" y2="90.17" width="0.889" layer="16"/>
-</signal>
-<signal name="SPEED2-" class="2">
-<contactref element="X5" pad="2"/>
-<contactref element="PL1" pad="13"/>
-<wire x1="33.1216" y1="29.0576" x2="33.1216" y2="12.8016" width="0.889" layer="16"/>
-<wire x1="33.7312" y1="29.6672" x2="33.1216" y2="29.0576" width="0.889" layer="16"/>
-<wire x1="33.7312" y1="69.088" x2="33.7312" y2="29.6672" width="0.889" layer="16"/>
-<wire x1="12.8016" y1="90.0176" x2="33.7312" y2="69.088" width="0.889" layer="16"/>
-<wire x1="33.1216" y1="12.8016" x2="33.02" y2="12.7" width="0.889" layer="16"/>
-<wire x1="12.8016" y1="90.0176" x2="12.7" y2="90.17" width="0.889" layer="16"/>
+<contactref element="D4" pad="A"/>
+<wire x1="30.48" y1="66.04" x2="27.94" y2="66.04" width="0.889" layer="1"/>
+<wire x1="27.94" y1="66.04" x2="25.4" y2="68.58" width="0.889" layer="1"/>
+<wire x1="25.4" y1="68.58" x2="14.0208" y2="68.58" width="0.889" layer="1"/>
 </signal>
 <signal name="N$2" class="1">

Commit message: Aggiornato frontend
Parts:
- added U$1: (no value), ITEM_Loghi:BASSA
- added U$2: (no value), ITEM_Loghi:UDINE
- added U$3: (no value), ITEM_Loghi:DANIELI
- D1: device diode:SMB -> diode:DO35Z10
- moved R5 121.7 mm to (142.9, 57.8)
- moved R1 91.6 mm to (141.0, 24.4), turned to 270 degrees
- moved LED1 81.9 mm to (135.3, 25.4), turned to 180 degrees
- moved OK1 14.5 mm to (135.3, 61.6)
- moved U3 10.0 mm to (29.2, 39.4)
- moved D1 7.65 mm to (139.1, 70.5)
- moved R2 7.10 mm to (142.9, 79.4), turned to 0 degrees
- moved R4 6.38 mm to (142.9, 65.4), turned to 180 degrees
- moved SV1 5.85 mm to (68.6, 26.7)
- moved SV2 4.62 mm to (87.6, 26.7)
- moved LED2 4.49 mm to (135.3, 74.9), turned to 180 degrees
- moved D3 4.02 mm to (20.3, 73.7)
- moved D4 3.86 mm to (20.3, 66.7)
- moved D2 2.29 mm to (44.5, 73.7)
- moved D5 2.01 mm to (44.5, 66.7)
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Connections:
- net +3V3: now also U3.2; no longer U3.VCC
- net GND: now also U3.1; no longer U3.GND
- net I2C_SCL: now also U3.3; no longer U3.SCL
- net I2C_SDA: now also U3.4; no longer U3.SDA
Routing:
- net +3V3: track 48.6 -> 160.2 mm, vias 0 -> 1
- net GND: track 261.1 -> 351.1 mm
- net SPEED1+: track 148.4 -> 96.0 mm, vias 0 -> 1
- net EXT_+5V: track 135.8 -> 118.9 mm, vias 1 -> 0
- net AUX_DIN: track 151.6 -> 135.6 mm
- net TORQUE2+: track 114.8 -> 101.6 mm
- net N$5: track 39.4 -> 26.3 mm
- net I2C_SCL: track 68.7 -> 59.6 mm, vias 0 -> 1
- net ACCEL1+: track 98.8 -> 106.5 mm
- net ACCEL0+: track 98.9 -> 106.5 mm
- net TORQUE1+: track 101.7 -> 94.3 mm, vias 0 -> 1
- net I2C_SDA: track 51.7 -> 44.7 mm
- net SPEED2+: track 120.3 -> 114.2 mm, vias 0 -> 1
- net RTD1_F+: track 60.4 -> 66.4 mm
- net RTD1_IN+: track 59.3 -> 65.3 mm
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Other:
- board text added: "DANIELI BUTTRIO"
- board text added: "ISIS BASSA FRIULANA"
- board text added: "ISIS MALIGNANI"
- board text added: "PROGETTO ITEM - A.S.2022-23"
