File: item_2022_Frontend_02_V7.sch (EAGLE design)
At the start: 29 parts, among them K1 351, U3 SSD1306_128X64, X1 MSTBA2, X10 MSTBA2, X11 MSTBA2, X12 MSTBA2, X13 MSTBA2, X14 MSTBA2, X15 MSTBA2, X2 MSTBA2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

Commit message: spostati BZW su Frontend da motherboard
Parts:
- added D2, D3, D4, D5: BZW06-10B, diode_LargePads:BZW04XXB
Connections:
- removed net SPEED1-: PL1.11, X4-2.1
- removed net SPEED2-: PL1.13, X5-2.1
- removed net TORQUE1-: PL1.7, X2-2.1
- removed net TORQUE2-: PL1.9, X3-2.1
- net GND: now also D2.2, D3.2, D4.2, D5.2, PL1.11, PL1.13, PL1.7, PL1.9, X2-2.1, X3-2.1, X4-2.1, X5-2.1
- net SPEED1+: now also D3.1
- net SPEED2+: now also D4.1
- net TORQUE1+: now also D5.1
- net TORQUE2+: now also D2.1
Changed lines of the file:
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@@
 <setting verticaltext="up"/>
 </settings>
-<grid distance="0.1" unitdist="inch" unit="inch" style="lines" multiple="1" display="no" altdistance="0.01" altunitdist="inch" altunit="inch"/>
+<grid distance="0.05" unitdist="inch" unit="inch" style="lines" multiple="2" display="yes" altdistance="0.01" altunitdist="inch" altunit="inch"/>
 <layers>
 <layer number="1" name="Top" color="4" fill="1" visible="no" active="no"/>
@@
 <part name="X21" library="con-phoenix-508" deviceset="MSTBA4" device=""/>
 <part name="PL1" library="con-harting-h" deviceset="16H" device=""/>
+<part name="D2" library="diode_LargePads" deviceset="BZW04XXB" device="" value="BZW06-10B"/>
+<part name="D3" library="diode_LargePads" deviceset="BZW04XXB" device="" value="BZW06-10B"/>
+<part name="D4" library="diode_LargePads" deviceset="BZW04XXB" device="" value="BZW06-10B"/>
+<part name="D5" library="diode_LargePads" deviceset="BZW04XXB" device="" value="BZW06-10B"/>
+<part name="GND4" library="supply1" deviceset="GND" device=""/>
+<part name="GND5" library="supply1" deviceset="GND" device=""/>
+<part name="GND6" library="supply1" deviceset="GND" device=""/>
 </parts>
 <sheets>
@@
 <instance part="PL1" gate="G$1" x="152.4" y="45.72" rot="R180"/>
 <instance part="K1" gate="3" x="91.44" y="149.86" rot="R270"/>
+<instance part="D2" gate="1" x="121.92" y="203.2" smashed="yes" rot="R270">
+<attribute name="NAME" x="123.825" y="204.47" size="1.778" layer="95" rot="R270"/>
+<attribute name="VALUE" x="118.491" y="204.47" size="1.778" layer="96" rot="R270"/>
+</instance>
+<instance part="D3" gate="1" x="129.54" y="203.2" smashed="yes" rot="R270">
+<attribute name="NAME" x="131.445" y="204.47" size="1.778" layer="95" rot="R270"/>
+<attribute name="VALUE" x="126.111" y="204.47" size="1.778" layer="96" rot="R270"/>
+</instance>
+<instance part="D4" gate="1" x="137.16" y="203.2" smashed="yes" rot="R270">
+<attribute name="NAME" x="139.065" y="204.47" size="1.778" layer="95" rot="R270"/>
+<attribute name="VALUE" x="133.731" y="204.47" size="1.778" layer="96" rot="R270"/>
+</instance>
+<instance part="D5" gate="1" x="114.3" y="203.2" smashed="yes" rot="R270">
+<attribute name="NAME" x="116.205" y="204.47" size="1.778" layer="95" rot="R270"/>
+<attribute name="VALUE" x="110.871" y="204.47" size="1.778" layer="96" rot="R270"/>
+</instance>
+<instance part="GND4" gate="1" x="73.66" y="182.88" smashed="yes">
+<attribute name="VALUE" x="71.12" y="180.34" size="1.778" layer="96"/>
+</instance>
+<instance part="GND5" gate="1" x="114.3" y="182.88" smashed="yes">
+<attribute name="VALUE" x="111.76" y="180.34" size="1.778" layer="96"/>
+</instance>
+<instance part="GND6" gate="1" x="142.24" y="25.4" smashed="yes">
+<attribute name="VALUE" x="139.7" y="22.86" size="1.778" layer="96"/>
+</instance>
 </instances>
 <busses>
@@
 <wire x1="307.34" y1="93.98" x2="307.34" y2="86.36" width="0.1524" layer="91"/>
 </segment>
+<segment>
+<pinref part="X5" gate="-2" pin="1"/>
+<pinref part="GND4" gate="1" pin="GND"/>
+<wire x1="73.66" y1="187.96" x2="71.12" y2="187.96" width="0.1524" layer="91"/>
+<wire x1="73.66" y1="185.42" x2="73.66" y2="187.96" width="0.1524" layer="91"/>
+<junction x="73.66" y="187.96"/>
+<pinref part="X4" gate="-2" pin="1"/>
+<wire x1="73.66" y1="203.2" x2="71.12" y2="203.2" width="0.1524" layer="91"/>
+<wire x1="73.66" y1="187.96" x2="73.66" y2="203.2" width="0.1524" layer="91"/>
+<junction x="73.66" y="203.2"/>
+<pinref part="X3" gate="-2" pin="1"/>
+<wire x1="73.66" y1="218.44" x2="71.12" y2="218.44" width="0.1524" layer="91"/>
+<wire x1="73.66" y1="203.2" x2="73.66" y2="218.44" width="0.1524" layer="91"/>
+<junction x="73.66" y="218.44"/>
+<pinref part="X2" gate="-2" pin="1"/>
+<wire x1="73.66" y1="233.68" x2="71.12" y2="233.68" width="0.1524" layer="91"/>
+<wire x1="73.66" y1="218.44" x2="73.66" y2="233.68" width="0.1524" layer="91"/>
+</segment>
+<segment>
+<pinref part="GND5" gate="1" pin="GND"/>
+<pinref part="D5" gate="1" pin="2"/>
+<wire x1="114.3" y1="185.42" x2="114.3" y2="187.96" width="0.1524" layer="91"/>
+<wire x1="114.3" y1="187.96" x2="114.3" y2="198.12" width="0.1524" layer="91"/>
+<wire x1="114.3" y1="187.96" x2="121.92" y2="187.96" width="0.1524" layer="91"/>
+<junction x="114.3" y="187.96"/>
+<pinref part="D4" gate="1" pin="2"/>
+<wire x1="121.92" y1="187.96" x2="129.54" y2="187.96" width="0.1524" layer="91"/>
+<wire x1="129.54" y1="187.96" x2="137.16" y2="187.96" width="0.1524" layer="91"/>
+<wire x1="137.16" y1="187.96" x2="137.16" y2="198.12" width="0.1524" layer="91"/>
+<pinref part="D3" gate="1" pin="2"/>
+<wire x1="129.54" y1="198.12" x2="129.54" y2="187.96" width="0.1524" layer="91"/>
+<junction x="129.54" y="187.96"/>
+<pinref part="D2" gate="1" pin="2"/>
+<wire x1="121.92" y1="198.12" x2="121.92" y2="187.96" width="0.1524" layer="91"/>
+<junction x="121.92" y="187.96"/>
+</segment>
+<segment>
+<pinref part="GND6" gate="1" pin="GND"/>
+<wire x1="142.24" y1="27.94" x2="142.24" y2="38.1" width="0.1524" layer="91"/>
+<pinref part="PL1" gate="G$1" pin="7"/>
+<wire x1="142.24" y1="38.1" x2="142.24" y2="40.64" width="0.1524" layer="91"/>
+<wire x1="142.24" y1="40.64" x2="142.24" y2="43.18" width="0.1524" layer="91"/>
+<wire x1="142.24" y1="43.18" x2="142.24" y2="45.72" width="0.1524" layer="91"/>
+<wire x1="142.24" y1="45.72" x2="144.78" y2="45.72" width="0.1524" layer="91"/>
+<pinref part="PL1" gate="G$1" pin="9"/>
+<wire x1="144.78" y1="43.18" x2="142.24" y2="43.18" width="0.1524" layer="91"/>
+<junction x="142.24" y="43.18"/>
+<pinref part="PL1" gate="G$1" pin="11"/>
+<wire x1="144.78" y1="40.64" x2="142.24" y2="40.64" width="0.1524" layer="91"/>
+<junction x="142.24" y="40.64"/>
+<pinref part="PL1" gate="G$1" pin="13"/>
+<wire x1="144.78" y1="38.1" x2="142.24" y2="38.1" width="0.1524" layer="91"/>
+<junction x="142.24" y="38.1"/>
+</segment>
 </net>
 <net name="I2C_SCL" class="0">
@@
 <pinref part="X2" gate="-1" pin="1"/>
 </segment>
+<segment>
+<pinref part="D5" gate="1" pin="1"/>
+<wire x1="114.3" y1="205.74" x2="114.3" y2="226.06" width="0.1524" layer="91"/>
+<wire x1="114.3" y1="226.06" x2="111.76" y2="226.06" width="0.1524" layer="91"/>
+<wire x1="116.84" y1="226.06" x2="114.3" y2="226.06" width="0.1524" layer="91"/>
+<junction x="114.3" y="226.06"/>
+<label x="116.84" y="226.06" size="1.4224" layer="95"/>
+</segment>
 </net>
 <net name="TORQUE2+" class="2">
@@
 <pinref part="X3" gate="-1" pin="1"/>
 </segment>
-</net>
-<net name="TORQUE1-" class="2">
-<segment>
-<wire x1="139.7" y1="45.72" x2="144.78" y2="45.72" width="0.1524" layer="91"/>
-<label x="129.54" y="45.72" size="1.4224" layer="95"/>
-<pinref part="PL1" gate="G$1" pin="7"/>
-</segment>
-<segment>
-<wire x1="76.2" y1="233.68" x2="71.12" y2="233.68" width="0.1524" layer="91"/>
-<label x="76.2" y="233.68" size="1.4224" layer="95"/>
-<pinref part="X2" gate="-2" pin="1"/>
-</segment>
-</net>
-<net name="TORQUE2-" class="2">
-<segment>
-<wire x1="139.7" y1="43.18" x2="144.78" y2="43.18" width="0.1524" layer="91"/>
-<label x="129.54" y="43.18" size="1.4224" layer="95"/>
-<pinref part="PL1" gate="G$1" pin="9"/>
-</segment>
-<segment>
-<wire x1="76.2" y1="218.44" x2="71.12" y2="218.44" width="0.1524" layer="91"/>
-<label x="76.2" y="218.44" size="1.4224" layer="95"/>
-<pinref part="X3" gate="-2" pin="1"/>
+<segment>
+<pinref part="D2" gate="1" pin="1"/>
+<wire x1="121.92" y1="205.74" x2="121.92" y2="220.98" width="0.1524" layer="91"/>
+<wire x1="121.92" y1="220.98" x2="124.46" y2="220.98" width="0.1524" layer="91"/>
+<wire x1="119.38" y1="220.98" x2="121.92" y2="220.98" width="0.1524" layer="91"/>
+<junction x="121.92" y="220.98"/>
+<label x="124.46" y="220.98" size="1.4224" layer="95"/>
 </segment>
 </net>
@@
 <pinref part="X4" gate="-1" pin="1"/>
 </segment>
+<segment>
+<pinref part="D3" gate="1" pin="1"/>
+<wire x1="129.54" y1="205.74" x2="129.54" y2="215.9" width="0.1524" layer="91"/>
+<wire x1="129.54" y1="215.9" x2="127" y2="215.9" width="0.1524" layer="91"/>
+<wire x1="132.08" y1="215.9" x2="129.54" y2="215.9" width="0.1524" layer="91"/>
+<junction x="129.54" y="215.9"/>
+<label x="132.08" y="215.9" size="1.4224" layer="95"/>
+</segment>
 </net>
 <net name="SPEED2+" class="2">
@@
 <pinref part="X5" gate="-1" pin="1"/>
 </segment>
-</net>
-<net name="SPEED1-" class="2">
-<segment>
-<wire x1="139.7" y1="40.64" x2="144.78" y2="40.64" width="0.1524" layer="91"/>
-<label x="129.54" y="40.64" size="1.4224" layer="95"/>
-<pinref part="PL1" gate="G$1" pin="11"/>
-</segment>
-<segment>
-<wire x1="76.2" y1="203.2" x2="71.12" y2="203.2" width="0.1524" layer="91"/>
-<label x="76.2" y="203.2" size="1.4224" layer="95"/>
-<pinref part="X4" gate="-2" pin="1"/>
-</segment>
-</net>
-<net name="SPEED2-" class="2">
-<segment>
-<wire x1="139.7" y1="38.1" x2="144.78" y2="38.1" width="0.1524" layer="91"/>
-<label x="129.54" y="38.1" size="1.4224" layer="95"/>
-<pinref part="PL1" gate="G$1" pin="13"/>
-</segment>
-<segment>
-<wire x1="76.2" y1="187.96" x2="71.12" y2="187.96" width="0.1524" layer="91"/>
-<label x="76.2" y="187.96" size="1.4224" layer="95"/>
-<pinref part="X5" gate="-2" pin="1"/>
-</segment>
-</net>
+<segment>
+<pinref part="D4" gate="1" pin="1"/>
+<wire x1="137.16" y1="210.82" x2="137.16" y2="205.74" width="0.1524" layer="91"/>
+<wire x1="139.7" y1="210.82" x2="137.16" y2="210.82" width="0.1524" layer="91"/>
+<wire x1="134.62" y1="210.82" x2="137.16" y2="210.82" width="0.1524" layer="91"/>
+<junction x="137.16" y="210.82"/>
+<label x="139.7" y="210.82" size="1.4224" layer="95"/>
+</segment>
+</net>

Commit message: Aggiornato frontend
Parts:
- D1: device diode:ZENER-DIODESMB -> diode:ZENER-DIODEDO35Z10
Other:
- moved on the sheet: U3
Changed lines of the file:
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@@
 <setting verticaltext="up"/>
 </settings>
-<grid distance="0.05" unitdist="inch" unit="inch" style="lines" multiple="2" display="yes" altdistance="0.01" altunitdist="inch" altunit="inch"/>
+<grid distance="0.05" unitdist="inch" unit="inch" style="lines" multiple="1" display="yes" altdistance="0.01" altunitdist="inch" altunit="inch"/>
 <layers>
-<layer number="1" name="Top" color="4" fill="1" visible="no" active="no"/>
-<layer number="2" name="Route2" color="1" fill="3" visible="no" active="no"/>
-<layer number="3" name="Route3" color="4" fill="3" visible="no" active="no"/>
-<layer number="14" name="Route14" color="1" fill="6" visible="no" active="no"/>
-<layer number="15" name="Route15" color="4" fill="6" visible="no" active="no"/>
-<layer number="16" name="Bottom" color="1" fill="1" visible="no" active="no"/>
-<layer number="17" name="Pads" color="2" fill="1" visible="no" active="no"/>
-<layer number="18" name="Vias" color="2" fill="1" visible="no" active="no"/>
-<layer number="19" name="Unrouted" color="6" fill="1" visible="no" active="no"/>
-<layer number="20" name="Dimension" color="15" fill="1" visible="no" active="no"/>
-<layer number="21" name="tPlace" color="7" fill="1" visible="no" active="no"/>
-<layer number="22" name="bPlace" color="7" fill="1" visible="no" active="no"/>
-<layer number="23" name="tOrigins" color="15" fill="1" visible="no" active="no"/>
-<layer number="24" name="bOrigins" color="15" fill="1" visible="no" active="no"/>
-<layer number="25" name="tNames" color="7" fill="1" visible="no" active="no"/>
-<layer number="26" name="bNames" color="7" fill="1" visible="no" active="no"/>
-<layer number="27" name="tValues" color="7" fill="1" visible="no" active="no"/>
-<layer number="28" name="bValues" color="7" fill="1" visible="no" active="no"/>
+<layer number="1" name="Top" color="4" fill="1" visible="yes" active="no"/>
+<layer number="2" name="Route2" color="1" fill="3" visible="yes" active="no"/>
+<layer number="3" name="Route3" color="4" fill="3" visible="yes" active="no"/>
+<layer number="14" name="Route14" color="1" fill="6" visible="yes" active="no"/>
+<layer number="15" name="Route15" color="4" fill="6" visible="yes" active="no"/>
+<layer number="16" name="Bottom" color="1" fill="1" visible="yes" active="no"/>
+<layer number="17" name="Pads" color="2" fill="1" visible="yes" active="no"/>
+<layer number="18" name="Vias" color="2" fill="1" visible="yes" active="no"/>
+<layer number="19" name="Unrouted" color="6" fill="1" visible="yes" active="no"/>
+<layer number="20" name="Dimension" color="15" fill="1" visible="yes" active="no"/>
+<layer number="21" name="tPlace" color="7" fill="1" visible="yes" active="no"/>
+<layer number="22" name="bPlace" color="7" fill="1" visible="yes" active="no"/>
+<layer number="23" name="tOrigins" color="15" fill="1" visible="yes" active="no"/>
+<layer number="24" name="bOrigins" color="15" fill="1" visible="yes" active="no"/>
+<layer number="25" name="tNames" color="7" fill="1" visible="yes" active="no"/>
+<layer number="26" name="bNames" color="7" fill="1" visible="yes" active="no"/>
+<layer number="27" name="tValues" color="7" fill="1" visible="yes" active="no"/>
+<layer number="28" name="bValues" color="7" fill="1" visible="yes" active="no"/>
 <layer number="29" name="tStop" color="7" fill="3" visible="no" active="no"/>
 <layer number="30" name="bStop" color="7" fill="6" visible="no" active="no"/>
@@
 <layer number="35" name="tGlue" color="7" fill="4" visible="no" active="no"/>
 <layer number="36" name="bGlue" color="7" fill="5" visible="no" active="no"/>
-<layer number="37" name="tTest" color="7" fill="1" visible="no" active="no"/>
-<layer number="38" name="bTest" color="7" fill="1" visible="no" active="no"/>
+<layer number="37" name="tTest" color="7" fill="1" visible="yes" active="no"/>
+<layer number="38" name="bTest" color="7" fill="1" visible="yes" active="no"/>
 <layer number="39" name="tKeepout" color="4" fill="11" visible="no" active="no"/>
 <layer number="40" name="bKeepout" color="1" fill="11" visible="no" active="no"/>
@@
 <layer number="44" name="Drills" color="7" fill="1" visible="no" active="no"/>
 <layer number="45" name="Holes" color="7" fill="1" visible="no" active="no"/>
-<layer number="46" name="Milling" color="3" fill="1" visible="no" active="no"/>
-<layer number="47" name="Measures" color="7" fill="1" visible="no" active="no"/>
-<layer number="48" name="Document" color="7" fill="1" visible="no" active="no"/>
-<layer number="49" name="Reference" color="7" fill="1" visible="no" active="no"/>
-<layer number="51" name="tDocu" color="7" fill="1" visible="no" active="no"/>
-<layer number="52" name="bDocu" color="7" fill="1" visible="no" active="no"/>
+<layer number="46" name="Milling" color="3" fill="1" visible="yes" active="no"/>
+<layer number="47" name="Measures" color="7" fill="1" visible="yes" active="no"/>
+<layer number="48" name="Document" color="7" fill="1" visible="yes" active="no"/>
+<layer number="49" name="Reference" color="7" fill="1" visible="yes" active="no"/>
+<layer number="51" name="tDocu" color="7" fill="1" visible="yes" active="no"/>
+<layer number="52" name="bDocu" color="7" fill="1" visible="yes" active="no"/>
 <layer number="88" name="SimResults" color="9" fill="1" visible="yes" active="yes"/>
 <layer number="89" name="SimProbes" color="9" fill="1" visible="yes" active="yes"/>
@@
 <parts>
 <part name="FRAME1" library="frames" deviceset="A3L-LOC" device=""/>
-<part name="U3" library="ssd1306oled" deviceset="SSD1306_128X64" device=""/>
 <part name="GND10" library="supply1" deviceset="GND" device=""/>
 <part name="+3V5" library="supply1" deviceset="+3V3" device=""/>
@@
 <part name="K1" library="relay" deviceset="351" device=""/>
 <part name="GND2" library="supply1" deviceset="GND" device=""/>
-<part name="D1" library="diode" deviceset="ZENER-DIODE" device="SMB" value="24V"/>
+<part name="D1" library="diode" deviceset="ZENER-DIODE" device="DO35Z10" value="24V"/>
 <part name="R2" library="rcl" deviceset="R-EU_" device="R0805" value="330"/>
 <part name="LED2" library="led" deviceset="LED" device="5MM"/>
@@
 <part name="GND5" library="supply1" deviceset="GND" device=""/>
 <part name="GND6" library="supply1" deviceset="GND" device=""/>
+<part name="U3" library="ssd1306oled" deviceset="SSD1306_128X64" device=""/>
 </parts>
 <sheets>
@@
 <attribute name="SHEET" x="357.505" y="5.08" size="2.54" layer="94"/>
 </instance>
-<instance part="U3" gate="G$1" x="226.06" y="43.18" smashed="yes">
-<attribute name="NAME" x="218.44" y="52.07" size="1.27" layer="95"/>
-<attribute name="VALUE" x="218.44" y="35.56" size="1.27" layer="95"/>
-</instance>
 <instance part="GND10" gate="1" x="210.82" y="33.02" smashed="yes">
 <attribute name="VALUE" x="208.28" y="30.48" size="1.778" layer="96"/>
@@
 <attribute name="VALUE" x="139.7" y="22.86" size="1.778" layer="96"/>
 </instance>
+<instance part="U3" gate="G$1" x="223.52" y="43.18"/>
 </instances>
 <busses>
@@
 <segment>
 <wire x1="210.82" y1="53.34" x2="210.82" y2="43.18" width="0.1524" layer="91"/>
+<pinref part="+3V5" gate="G$1" pin="+3V3"/>
 <pinref part="U3" gate="G$1" pin="VCC"/>
-<wire x1="210.82" y1="43.18" x2="215.9" y2="43.18" width="0.1524" layer="91"/>
-<pinref part="+3V5" gate="G$1" pin="+3V3"/>
+<wire x1="213.36" y1="43.18" x2="210.82" y2="43.18" width="0.1524" layer="91"/>
 </segment>
 <segment>
@@
 <label x="165.1" y="38.1" size="1.4224" layer="95"/>
 <pinref part="PL1" gate="G$1" pin="14"/>
-</segment>
-<segment>
-<pinref part="U3" gate="G$1" pin="GND"/>
-<wire x1="215.9" y1="40.64" x2="210.82" y2="40.64" width="0.1524" layer="91"/>
-<wire x1="210.82" y1="40.64" x2="210.82" y2="35.56" width="0.1524" layer="91"/>
-<pinref part="GND10" gate="1" pin="GND"/>
 </segment>
 <segment>
@@
 <junction x="142.24" y="38.1"/>
 </segment>
+<segment>
+<pinref part="U3" gate="G$1" pin="GND"/>
+<pinref part="GND10" gate="1" pin="GND"/>
+<wire x1="213.36" y1="40.64" x2="210.82" y2="40.64" width="0.1524" layer="91"/>
+<wire x1="210.82" y1="40.64" x2="210.82" y2="35.56" width="0.1524" layer="91"/>
+</segment>
 </net>
 <net name="I2C_SCL" class="0">
@@
 </segment>
 <segment>
+<label x="200.66" y="45.72" size="1.4224" layer="95"/>
 <pinref part="U3" gate="G$1" pin="SCL"/>
-<wire x1="205.74" y1="45.72" x2="215.9" y2="45.72" width="0.1524" layer="91"/>
-<label x="205.74" y="45.72" size="1.4224" layer="95"/>
+<wire x1="213.36" y1="45.72" x2="200.66" y2="45.72" width="0.1524" layer="91"/>
 </segment>
 </net>
@@
 </segment>
 <segment>
+<label x="200.66" y="48.26" size="1.4224" layer="95"/>
 <pinref part="U3" gate="G$1" pin="SDA"/>
-<wire x1="205.74" y1="48.26" x2="215.9" y2="48.26" width="0.1524" layer="91"/>
-<label x="205.74" y="48.26" size="1.4224" layer="95"/>
+<wire x1="213.36" y1="48.26" x2="200.66" y2="48.26" width="0.1524" layer="91"/>
 </segment>
 </net>
