File: item_2022_Frontend_02_V7.sch (EAGLE design)
At the start: 33 parts, among them K1 351, U3 SSD1306_128X64, X1 MSTBA2, X10 MSTBA2, X11 MSTBA2, X12 MSTBA2, X13 MSTBA2, X14 MSTBA2, X15 MSTBA2, X2 MSTBA2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

Commit message: FrontEnd con PE
Parts:
- added H1, H2: MOUNT-PAD-ROUND3.6, holes:MOUNT-PAD-ROUND3.6
- X6, X7: value MSTBA2 -> MSTBA3; device con-phoenix-508:MSTBA2 -> con-phoenix-508:MSTBA3
Connections:
- new net PE: H1.MOUNT, H2.MOUNT, X6-3.1, X7-3.1
Other:
- moved on the sheet: K1, X14-1, X14-2, X7-1, X7-2
Changed lines of the file:
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@@
 <setting verticaltext="up"/>
 </settings>
-<grid distance="0.1" unitdist="inch" unit="inch" style="lines" multiple="1" display="no" altdistance="0.01" altunitdist="inch" altunit="inch"/>
+<grid distance="0.1" unitdist="inch" unit="inch" style="lines" multiple="1" display="yes" altdistance="0.01" altunitdist="inch" altunit="inch"/>
 <layers>
 <layer number="1" name="Top" color="4" fill="1" visible="no" active="no"/>
@@
 <part name="X14" library="con-phoenix-508" deviceset="MSTBA2" device=""/>
 <part name="X15" library="con-phoenix-508" deviceset="MSTBA2" device=""/>
-<part name="X6" library="con-phoenix-508" deviceset="MSTBA2" device=""/>
-<part name="X7" library="con-phoenix-508" deviceset="MSTBA2" device=""/>
 <part name="X11" library="con-phoenix-508" deviceset="MSTBA2" device=""/>
 <part name="X13" library="con-phoenix-508" deviceset="MSTBA2" device=""/>
@@
 <part name="GND6" library="supply1" deviceset="GND" device=""/>
 <part name="U3" library="ssd1306oled" deviceset="SSD1306_128X64" device=""/>
+<part name="X6" library="con-phoenix-508" deviceset="MSTBA3" device=""/>
+<part name="X7" library="con-phoenix-508" deviceset="MSTBA3" device=""/>
+<part name="H1" library="holes" deviceset="MOUNT-PAD-ROUND" device="3.6"/>
+<part name="H2" library="holes" deviceset="MOUNT-PAD-ROUND" device="3.6"/>
 </parts>
 <sheets>
@@
 <text x="203.2" y="187.96" size="1.778" layer="97">Accel0+</text>
 <text x="203.2" y="182.88" size="1.778" layer="97">Accel0-</text>
-<text x="203.2" y="172.72" size="1.778" layer="97">Accel1+</text>
-<text x="203.2" y="167.64" size="1.778" layer="97">Accel1-</text>
+<text x="203.2" y="167.64" size="1.778" layer="97">Accel1+</text>
+<text x="203.2" y="162.56" size="1.778" layer="97">Accel1-</text>
 <text x="208.28" y="231.14" size="1.4224" layer="97" align="center-right">RTD1 - connettore
 verso sensore</text>
@@
 <wire x1="302.26" y1="198.12" x2="299.72" y2="195.58" width="0.254" layer="97"/>
 <wire x1="203.2" y1="190.5" x2="200.66" y2="187.96" width="0.254" layer="97"/>
-<wire x1="200.66" y1="187.96" x2="200.66" y2="167.64" width="0.254" layer="97"/>
-<wire x1="200.66" y1="167.64" x2="203.2" y2="165.1" width="0.254" layer="97"/>
+<wire x1="200.66" y1="187.96" x2="200.66" y2="157.48" width="0.254" layer="97"/>
+<wire x1="200.66" y1="157.48" x2="203.2" y2="154.94" width="0.254" layer="97"/>
 <text x="17.78" y="210.82" size="1.778" layer="97">Modulo esterno
 condizionamento
@@
 (Cavo coassiale ? )</text>
 <wire x1="12.7" y1="180.34" x2="172.72" y2="180.34" width="0.254" layer="97" style="shortdash"/>
-<wire x1="172.72" y1="99.06" x2="12.7" y2="99.06" width="0.254" layer="97" style="shortdash"/>
-<wire x1="12.7" y1="99.06" x2="12.7" y2="180.34" width="0.254" layer="97" style="shortdash"/>
-<text x="15.24" y="101.6" size="2.1844" layer="97">NOTA: qui vanno collegati i due alimentatori (+5v e +24V)
+<wire x1="172.72" y1="93.98" x2="12.7" y2="93.98" width="0.254" layer="97" style="shortdash"/>
+<wire x1="12.7" y1="93.98" x2="12.7" y2="180.34" width="0.254" layer="97" style="shortdash"/>
+<text x="15.24" y="96.52" size="2.1844" layer="97">NOTA: qui vanno collegati i due alimentatori (+5v e +24V)
 * Lasciamo i connettori X1 e X12 su questa scheda?
 * Altrimenti, il +24V lo facciamo arrivare solo alla scheda generatore di corrente?
@@
 * Il +5V ha senso farlo arrivare qui e collegare un interruttore On/Off per comandare l'accensione della ESP32.</text>
 <text x="281.94" y="43.18" size="1.4224" layer="97">On/Off</text>
-<text x="147.32" y="147.32" size="1.778" layer="97" align="center-left">Alla scheda
+<text x="139.7" y="147.32" size="1.778" layer="97" align="center-left">Alla scheda
 generatori
 di corrente</text>
-<wire x1="142.24" y1="152.4" x2="144.78" y2="149.86" width="0.254" layer="97"/>
-<wire x1="144.78" y1="149.86" x2="144.78" y2="144.78" width="0.254" layer="97"/>
-<wire x1="144.78" y1="144.78" x2="142.24" y2="142.24" width="0.254" layer="97"/>
-<wire x1="172.72" y1="180.34" x2="172.72" y2="99.06" width="0.254" layer="97" style="shortdash"/>
+<wire x1="134.62" y1="152.4" x2="137.16" y2="149.86" width="0.254" layer="97"/>
+<wire x1="137.16" y1="149.86" x2="137.16" y2="144.78" width="0.254" layer="97"/>
+<wire x1="137.16" y1="144.78" x2="134.62" y2="142.24" width="0.254" layer="97"/>
+<wire x1="172.72" y1="180.34" x2="172.72" y2="93.98" width="0.254" layer="97" style="shortdash"/>
 <text x="208.28" y="111.76" size="1.778" layer="97" align="center-right">Ingresso ausiliario
 da PLC, +24VDC</text>
@@
 <instance part="X12" gate="-1" x="66.04" y="149.86"/>
 <instance part="X12" gate="-2" x="66.04" y="144.78"/>
-<instance part="X14" gate="-1" x="124.46" y="149.86" rot="MR0"/>
-<instance part="X14" gate="-2" x="124.46" y="144.78" rot="MR0"/>
+<instance part="X14" gate="-1" x="116.84" y="149.86" rot="MR0"/>
+<instance part="X14" gate="-2" x="116.84" y="144.78" rot="MR0"/>
 <instance part="X15" gate="-1" x="226.06" y="114.3"/>
 <instance part="X15" gate="-2" x="226.06" y="109.22"/>
-<instance part="X6" gate="-1" x="226.06" y="187.96"/>
-<instance part="X6" gate="-2" x="226.06" y="182.88"/>
-<instance part="X7" gate="-1" x="226.06" y="172.72"/>
-<instance part="X7" gate="-2" x="226.06" y="167.64"/>
 <instance part="X11" gate="-1" x="292.1" y="187.96" rot="MR0"/>
 <instance part="X11" gate="-2" x="292.1" y="182.88" rot="MR0"/>
@@
 <instance part="X21" gate="-4" x="226.06" y="198.12"/>
 <instance part="PL1" gate="G$1" x="152.4" y="45.72" rot="R180"/>
-<instance part="K1" gate="3" x="91.44" y="149.86" rot="R270"/>
+<instance part="K1" gate="3" x="83.82" y="149.86" rot="R270"/>
 <instance part="D2" gate="1" x="121.92" y="203.2" smashed="yes" rot="R270">
 <attribute name="NAME" x="123.825" y="204.47" size="1.778" layer="95" rot="R270"/>
@@
 </instance>
 <instance part="U3" gate="G$1" x="223.52" y="43.18"/>
+<instance part="X6" gate="-1" x="226.06" y="187.96"/>
+<instance part="X6" gate="-2" x="226.06" y="182.88"/>
+<instance part="X6" gate="-3" x="226.06" y="177.8"/>
+<instance part="X7" gate="-1" x="226.06" y="167.64"/>
+<instance part="X7" gate="-2" x="226.06" y="162.56"/>
+<instance part="X7" gate="-3" x="226.06" y="157.48"/>
+<instance part="H1" gate="G$1" x="238.76" y="142.24"/>
+<instance part="H2" gate="G$1" x="238.76" y="132.08"/>
 </instances>
 <busses>
@@
 </segment>
 <segment>
-<wire x1="114.3" y1="144.78" x2="119.38" y2="144.78" width="0.1524" layer="91"/>
-<label x="109.22" y="144.78" size="1.4224" layer="95"/>
+<wire x1="106.68" y1="144.78" x2="111.76" y2="144.78" width="0.1524" layer="91"/>
+<label x="101.6" y="144.78" size="1.4224" layer="95"/>
 <pinref part="X14" gate="-2" pin="1"/>
 </segment>
@@
 <net name="ACCEL0+" class="2">
 <segment>
-<wire x1="236.22" y1="187.96" x2="231.14" y2="187.96" width="0.1524" layer="91"/>
 <label x="236.22" y="187.96" size="1.4224" layer="95"/>
 <pinref part="X6" gate="-1" pin="1"/>
+<wire x1="231.14" y1="187.96" x2="236.22" y2="187.96" width="0.1524" layer="91"/>
 </segment>
 <segment>
@@
 <net name="ACCEL0-" class="2">
 <segment>
-<wire x1="236.22" y1="182.88" x2="231.14" y2="182.88" width="0.1524" layer="91"/>
 <label x="236.22" y="182.88" size="1.4224" layer="95"/>
 <pinref part="X6" gate="-2" pin="1"/>
+<wire x1="231.14" y1="182.88" x2="236.22" y2="182.88" width="0.1524" layer="91"/>
 </segment>
 <segment>
@@
 <net name="ACCEL1+" class="2">
 <segment>
-<wire x1="236.22" y1="172.72" x2="231.14" y2="172.72" width="0.1524" layer="91"/>
-<label x="236.22" y="172.72" size="1.4224" layer="95"/>
+<label x="236.22" y="167.64" size="1.4224" layer="95"/>
 <pinref part="X7" gate="-1" pin="1"/>
+<wire x1="231.14" y1="167.64" x2="236.22" y2="167.64" width="0.1524" layer="91"/>
 </segment>
 <segment>
@@
 <net name="ACCEL1-" class="2">
 <segment>
-<wire x1="236.22" y1="167.64" x2="231.14" y2="167.64" width="0.1524" layer="91"/>
-<label x="236.22" y="167.64" size="1.4224" layer="95"/>
+<label x="236.22" y="162.56" size="1.4224" layer="95"/>
 <pinref part="X7" gate="-2" pin="1"/>
+<wire x1="231.14" y1="162.56" x2="236.22" y2="162.56" width="0.1524" layer="91"/>
 </segment>
 <segment>
@@
 <net name="+24VDC" class="1">
 <segment>
-<wire x1="106.68" y1="149.86" x2="119.38" y2="149.86" width="0.1524" layer="91"/>
-<label x="109.22" y="151.13" size="1.4224" layer="95"/>
+<wire x1="99.06" y1="149.86" x2="111.76" y2="149.86" width="0.1524" layer="91"/>
+<label x="101.6" y="151.13" size="1.4224" layer="95"/>
 <pinref part="X14" gate="-1" pin="1"/>
 <pinref part="K1" gate="3" pin="S"/>
-<wire x1="96.52" y1="154.94" x2="106.68" y2="154.94" width="0.1524" layer="91"/>
-<wire x1="106.68" y1="154.94" x2="106.68" y2="149.86" width="0.1524" layer="91"/>
+<wire x1="88.9" y1="154.94" x2="99.06" y2="154.94" width="0.1524" layer="91"/>
+<wire x1="99.06" y1="154.94" x2="99.06" y2="149.86" width="0.1524" layer="91"/>
 </segment>
 </net>
@@
 <pinref part="K1" gate="3" pin="P"/>
 <pinref part="X12" gate="-1" pin="1"/>
-<wire x1="88.9" y1="149.86" x2="71.12" y2="149.86" width="0.1524" layer="91"/>
-</segment>
-</net>
+<wire x1="81.28" y1="149.86" x2="71.12" y2="149.86" width="0.1524" layer="91"/>
+</segment>
+</net>
+<net name="PE" class="1">
+<segment>
+<pinref part="X6" gate="-3" pin="1"/>
+<wire x1="231.14" y1="177.8" x2="233.68" y2="177.8" width="0.1524" layer="91"/>
+<wire x1="233.68" y1="177.8" x2="233.68" y2="157.48" width="0.1524" layer="91"/>
+<pinref part="X7" gate="-3" pin="1"/>
+<wire x1="233.68" y1="157.48" x2="231.14" y2="157.48" width="0.1524" layer="91"/>
+<junction x="233.68" y="157.48"/>
+<pinref part="H2" gate="G$1" pin="MOUNT"/>
+<wire x1="236.22" y1="132.08" x2="233.68" y2="132.08" width="0.1524" layer="91"/>
+<wire x1="233.68" y1="132.08" x2="233.68" y2="142.24" width="0.1524" layer="91"/>
+<pinref part="H1" gate="G$1" pin="MOUNT"/>
+<wire x1="233.68" y1="142.24" x2="233.68" y2="157.48" width="0.1524" layer="91"/>
+<wire x1="236.22" y1="142.24" x2="233.68" y2="142.24" width="0.1524" layer="91"/>
+<junction x="233.68" y="142.24"/>
+</segment>
+</net>
